File: scaler/a01_1.sch (KiCad schematic (older format))
At the start: 4 parts, among them U1028 74HC04, U1029 74HC02, U1030 74HC02, U1031 74HC02

Commit message: Added and tied in the Alarms module.
I've placed page 2 of Counter Cell 2 here as page 2 of alarms. It didn't
fit in the counter cells, despite producing a few counter-related
signals -- and it mostly handles monitor stuff, which is a good fit for
what's going on here. As part of this I modernized the timer and scaler
connectors.

There seems to be lots of oscillations in the the simulation. Initial
conditions to correct those to follow.
Parts:
- added unit 5 of U1028
- added unit 6 of U1028
- added U1063: 74HC04, symbol 74HC04
Connections:
- net F05A: now also U1028.11
- net F05B: now also U1028.13
- net F07B: now also U1063.1
- net F10A: now also U1063.3
- net GND: now also U1028.7 (GND), U1028.7 (GND), U1063.7 (GND), U1063.7 (GND)
- net VCC: now also U1028.14 (VCC), U1028.14 (VCC), U1063.14 (VCC), U1063.14 (VCC)
- new net F05A/: U1028.10
- new net F05B/: U1028.12
- new net F07B/: U1063.2
- new net F10A/: U1063.4
Other:
- moved on the sheet: U1030A, U1030B, U1030C, U1030D, U1031A, U1031B, U1031C, U1031D

Commit message: Tied in Inout IV and renamed MONPCH to the original MON+CH
Parts:
- added unit 3 of U1063
- added unit 4 of U1063
- added unit 5 of U1063
Connections:
- net F09B: now also U1063.5
- net FS07: now also U1063.9
- net GND: now also U1063.7 (GND), U1063.7 (GND), U1063.7 (GND)
- net VCC: now also U1063.14 (VCC), U1063.14 (VCC), U1063.14 (VCC)
- new net F09B/: U1063.6
- new net FS07/: U1063.11, U1063.8
- new net FS07A: U1063.10
Other:
- moved on the sheet: U1063A
Changed lines of the file:
@@
 	14200 2000 14750 2000
 Wire Wire Line
-	14200 2250 14350 2250
-Text HLabel 14350 2250 2    60   Output ~ 0
+	14200 2250 14550 2250
+Text HLabel 14550 2250 2    60   Output ~ 0
 F07B
 Text HLabel 14350 1900 2    60   Output ~ 0
@@
 L 74HC04 U1063
 U 1 1 57C58ED9
-P 14800 2700
-F 0 "U1063" H 14950 2800 40  0000 C CNN
-F 1 "74HC04" H 15000 2600 40  0000 C CNN
-F 2 "" H 14800 2700 60  0000 C CNN
-F 3 "" H 14800 2700 60  0000 C CNN
-	1    14800 2700
-	1    0    0    -1
-$EndComp
-Wire Wire Line
-	14300 2250 14300 2700
-Wire Wire Line
-	14300 2700 14350 2700
-Wire Wire Line
-	15250 2700 15350 2700
-Text HLabel 15350 2700 2    60   Output ~ 0
+P 15100 2650
+F 0 "U1063" H 15250 2750 40  0000 C CNN
+F 1 "74HC04" H 15300 2550 40  0000 C CNN
+F 2 "" H 15100 2650 60  0000 C CNN
+F 3 "" H 15100 2650 60  0000 C CNN
+	1    15100 2650
+	1    0    0    -1
+$EndComp
+Wire Wire Line
+	14500 2250 14500 2650
+Wire Wire Line
+	14500 2650 14650 2650
+Wire Wire Line
+	15550 2650 15600 2650
+Text HLabel 15600 2650 2    60   Output ~ 0
 F07B/
-Connection ~ 14300 2250
+Connection ~ 14500 2250
 $Comp
 L 74HC04 U1063
@@
 Text HLabel 5200 5300 2    60   Output ~ 0
 F10A/
+$Comp
+L 74HC04 U1063
+U 3 1 5715108F
+P 19700 2700
+F 0 "U1063" H 19850 2800 40  0000 C CNN
+F 1 "74HC04" H 19900 2600 40  0000 C CNN
+F 2 "" H 19700 2700 60  0000 C CNN
+F 3 "" H 19700 2700 60  0000 C CNN
+	3    19700 2700
+	1    0    0    -1
+$EndComp
+Wire Wire Line
+	18600 2250 18600 2700
+Wire Wire Line
+	18600 2700 19250 2700
+Wire Wire Line
+	20150 2700 20200 2700
+Text HLabel 20200 2700 2    60   Output ~ 0
+F09B/
+Connection ~ 18600 2250
+Wire Wire Line
+	14300 1900 14300 3000
+Wire Wire Line
+	14300 3000 14350 3000
+Connection ~ 14300 1900
+$Comp
+L 74HC04 U1063
+U 4 1 5717DE56
+P 14800 3000
+F 0 "U1063" H 14950 3100 40  0000 C CNN
+F 1 "74HC04" H 15000 2900 40  0000 C CNN
+F 2 "" H 14800 3000 60  0000 C CNN
+F 3 "" H 14800 3000 60  0000 C CNN
+	4    14800 3000
+	1    0    0    -1
+$EndComp
+Wire Wire Line
+	15250 3000 15600 3000
+$Comp
+L 74HC04 U1063
+U 5 1 571850AF
+P 16050 3000
+F 0 "U1063" H 16200 3100 40  0000 C CNN
+F 1 "74HC04" H 16250 2900 40  0000 C CNN
+F 2 "" H 16050 3000 60  0000 C CNN
+F 3 "" H 16050 3000 60  0000 C CNN
+	5    16050 3000
+	1    0    0    -1
+$EndComp
+Wire Wire Line
+	16500 3000 16550 3000
+Text HLabel 16550 3000 2    60   Output ~ 0
+FS07A
+Wire Wire Line
+	15300 3000 15300 2900
+Wire Wire Line
+	15300 2900 15350 2900
+Connection ~ 15300 3000
+Text HLabel 15350 2900 2    60   Output ~ 0
+FS07/
 $EndSCHEMATC

Commit message: Tied in Inout II.
Parts:
- added unit 6 of U1063
Connections:
- net FS05: now also U1063.13
- net GND: now also U1063.7 (GND)
- net VCC: now also U1063.14 (VCC)
- new net FS05/: U1063.12
Other:
- moved on the sheet: U1028D
Changed lines of the file:
@@
 	10550 1900 11050 1900
 Wire Wire Line
-	10450 2000 10450 1400
-Wire Wire Line
-	10450 1400 10550 1400
+	10450 2000 10450 1550
+Wire Wire Line
+	10450 1550 10550 1550
 Text HLabel 10650 2150 2    60   Output ~ 0
 F05A
@@
 L 74HC04 U1028
 U 4 1 5633EC7D
-P 11000 1400
-F 0 "U1028" H 11150 1500 40  0000 C CNN
-F 1 "74HC04" H 11200 1300 40  0000 C CNN
-F 2 "" H 11000 1400 60  0000 C CNN
-F 3 "" H 11000 1400 60  0000 C CNN
-	4    11000 1400
+P 11000 1550
+F 0 "U1028" H 11150 1650 40  0000 C CNN
+F 1 "74HC04" H 11200 1450 40  0000 C CNN
+F 2 "" H 11000 1550 60  0000 C CNN
+F 3 "" H 11000 1550 60  0000 C CNN
+	4    11000 1550
 	1    0    0    -1
 $EndComp
@@
 FS04A
 Wire Wire Line
-	11450 1400 11550 1400
-Text HLabel 11550 1400 2    60   Output ~ 0
+	11450 1550 11550 1550
+Text HLabel 11550 1550 2    60   Output ~ 0
 FS05A
 Wire Wire Line
@@
 Text HLabel 15350 2900 2    60   Output ~ 0
 FS07/
+$Comp
+L 74HC04 U1063
+U 6 1 57B92C58
+P 10500 1300
+F 0 "U1063" H 10650 1400 40  0000 C CNN
+F 1 "74HC04" H 10700 1200 40  0000 C CNN
+F 2 "" H 10500 1300 60  0000 C CNN
+F 3 "" H 10500 1300 60  0000 C CNN
+	6    10500 1300
+	1    0    0    -1
+$EndComp
+Wire Wire Line
+	10000 1900 10000 1300
+Wire Wire Line
+	10000 1300 10050 1300
+Connection ~ 10000 1900
+Wire Wire Line
+	10950 1300 11050 1300
+Text HLabel 11050 1300 2    60   Output ~ 0
+FS05/
 $EndSCHEMATC

Commit message: Added most of the rest of Inout III and tied it in. Still not sure where to put the downlink stuff, standby, and CHOR propers.
Parts:
- added U1064: 74HC04, symbol 74HC04
Connections:
- net FS09: now also U1064.1
- net GND: now also U1064.7 (GND)
- net VCC: now also U1064.14 (VCC)
- new net FS09/: U1064.2
Changed lines of the file:
@@
 	18500 2000 19050 2000
 Wire Wire Line
-	18500 2250 18650 2250
-Text HLabel 18650 2250 2    60   Output ~ 0
+	18500 2250 18800 2250
+Text HLabel 18800 2250 2    60   Output ~ 0
 F09B
 Text HLabel 18650 1900 2    60   Output ~ 0
@@
 $EndComp
 Wire Wire Line
-	18600 2250 18600 2700
-Wire Wire Line
-	18600 2700 19250 2700
+	18750 2250 18750 2700
+Wire Wire Line
+	18750 2700 19250 2700
 Wire Wire Line
 	20150 2700 20200 2700
 Text HLabel 20200 2700 2    60   Output ~ 0
 F09B/
-Connection ~ 18600 2250
+Connection ~ 18750 2250
 Wire Wire Line
 	14300 1900 14300 3000
@@
 Text HLabel 11050 1300 2    60   Output ~ 0
 FS05/
+Wire Wire Line
+	18600 1900 18600 3100
+Wire Wire Line
+	18600 3100 19250 3100
+Connection ~ 18600 1900
+$Comp
+L 74HC04 U1064
+U 1 1 57219F28
+P 19700 3100
+F 0 "U1064" H 19850 3200 40  0000 C CNN
+F 1 "74HC04" H 19900 3000 40  0000 C CNN
+F 2 "" H 19700 3100 60  0000 C CNN
+F 3 "" H 19700 3100 60  0000 C CNN
+	1    19700 3100
+	1    0    0    -1
+$EndComp
+Wire Wire Line
+	20150 3100 20200 3100
+Text HLabel 20200 3100 2    60   Output ~ 0
+FS09/
 $EndSCHEMATC
