File: scaler/a01_2.sch (KiCad schematic (older format))
At the start: 4 parts, among them U1059 74HC02, U1060 74HC02, U1061 74HC02, U1062 74HC02

Commit message: SUPER BROKEN: Pulled in all NOR gates into the custom library, and changed the shape of 74HC04. Some, but not all, gates have standalone power pin parts. Scaler and Timer have been updated to use the new lib and rearranged to fit the new NOTs.
Changed lines of the file:
@@
 LIBS:linear
 LIBS:regul
-LIBS:74xx
+LIBS:agc_kicad_components
 LIBS:cmos4000
 LIBS:adc-dac
@@
 LIBS:contrib
 LIBS:valves
-LIBS:agc_kicad_components
 LIBS:scaler-cache
 EELAYER 25 0
@@
 P 12950 1700
 F 0 "U1060" H 12950 1750 60  0000 C CNN
-F 1 "74HC02" H 13000 1650 60  0000 C CNN
+F 1 "74HC02" H 13000 1650 60  0001 C CNN
 F 2 "" H 12950 1700 60  0000 C CNN
 F 3 "" H 12950 1700 60  0000 C CNN
@@
 P 15100 1700
 F 0 "U1060" H 15100 1750 60  0000 C CNN
-F 1 "74HC02" H 15150 1650 60  0000 C CNN
+F 1 "74HC02" H 15150 1650 60  0001 C CNN
 F 2 "" H 15100 1700 60  0000 C CNN
 F 3 "" H 15100 1700 60  0000 C CNN
@@
 P 17250 1700
 F 0 "U1060" H 17250 1750 60  0000 C CNN
-F 1 "74HC02" H 17300 1650 60  0000 C CNN
+F 1 "74HC02" H 17300 1650 60  0001 C CNN
 F 2 "" H 17250 1700 60  0000 C CNN
 F 3 "" H 17250 1700 60  0000 C CNN
@@
 P 19400 1700
 F 0 "U1060" H 19400 1750 60  0000 C CNN
-F 1 "74HC02" H 19450 1650 60  0000 C CNN
+F 1 "74HC02" H 19450 1650 60  0001 C CNN
 F 2 "" H 19400 1700 60  0000 C CNN
 F 3 "" H 19400 1700 60  0000 C CNN
@@
 P 4350 3800
 F 0 "U1061" H 4350 3850 60  0000 C CNN
-F 1 "74HC02" H 4400 3750 60  0000 C CNN
+F 1 "74HC02" H 4400 3750 60  0001 C CNN
 F 2 "" H 4350 3800 60  0000 C CNN
 F 3 "" H 4350 3800 60  0000 C CNN
@@
 P 6500 3800
 F 0 "U1061" H 6500 3850 60  0000 C CNN
-F 1 "74HC02" H 6550 3750 60  0000 C CNN
+F 1 "74HC02" H 6550 3750 60  0001 C CNN
 F 2 "" H 6500 3800 60  0000 C CNN
 F 3 "" H 6500 3800 60  0000 C CNN
@@
 P 8650 3800
 F 0 "U1061" H 8650 3850 60  0000 C CNN
-F 1 "74HC02" H 8700 3750 60  0000 C CNN
+F 1 "74HC02" H 8700 3750 60  0001 C CNN
 F 2 "" H 8650 3800 60  0000 C CNN
 F 3 "" H 8650 3800 60  0000 C CNN
@@
 P 10800 3800
 F 0 "U1061" H 10800 3850 60  0000 C CNN
-F 1 "74HC02" H 10850 3750 60  0000 C CNN
+F 1 "74HC02" H 10850 3750 60  0001 C CNN
 F 2 "" H 10800 3800 60  0000 C CNN
 F 3 "" H 10800 3800 60  0000 C CNN
@@
 P 12950 3800
 F 0 "U1062" H 12950 3850 60  0000 C CNN
-F 1 "74HC02" H 13000 3750 60  0000 C CNN
+F 1 "74HC02" H 13000 3750 60  0001 C CNN
 F 2 "" H 12950 3800 60  0000 C CNN
 F 3 "" H 12950 3800 60  0000 C CNN
@@
 P 15100 3800
 F 0 "U1062" H 15100 3850 60  0000 C CNN
-F 1 "74HC02" H 15150 3750 60  0000 C CNN
+F 1 "74HC02" H 15150 3750 60  0001 C CNN
 F 2 "" H 15100 3800 60  0000 C CNN
 F 3 "" H 15100 3800 60  0000 C CNN
@@
 P 17250 3800
 F 0 "U1062" H 17250 3850 60  0000 C CNN
-F 1 "74HC02" H 17300 3750 60  0000 C CNN
+F 1 "74HC02" H 17300 3750 60  0001 C CNN
 F 2 "" H 17250 3800 60  0000 C CNN
 F 3 "" H 17250 3800 60  0000 C CNN
@@
 P 19400 3800
 F 0 "U1062" H 19400 3850 60  0000 C CNN
-F 1 "74HC02" H 19450 3750 60  0000 C CNN
+F 1 "74HC02" H 19450 3750 60  0001 C CNN
 F 2 "" H 19400 3800 60  0000 C CNN
 F 3 "" H 19400 3800 60  0000 C CNN
@@
 P 4350 1700
 F 0 "U1059" H 4350 1750 60  0000 C CNN
-F 1 "74HC02" H 4400 1650 60  0000 C CNN
+F 1 "74HC02" H 4400 1650 60  0001 C CNN
 F 2 "" H 4350 1700 60  0000 C CNN
 F 3 "" H 4350 1700 60  0000 C CNN
@@
 P 6500 1700
 F 0 "U1059" H 6500 1750 60  0000 C CNN
-F 1 "74HC02" H 6550 1650 60  0000 C CNN
+F 1 "74HC02" H 6550 1650 60  0001 C CNN
 F 2 "" H 6500 1700 60  0000 C CNN
 F 3 "" H 6500 1700 60  0000 C CNN
@@
 P 8650 1700
 F 0 "U1059" H 8650 1750 60  0000 C CNN
-F 1 "74HC02" H 8700 1650 60  0000 C CNN
+F 1 "74HC02" H 8700 1650 60  0001 C CNN
 F 2 "" H 8650 1700 60  0000 C CNN
 F 3 "" H 8650 1700 60  0000 C CNN
@@
 P 10800 1700
 F 0 "U1059" H 10800 1750 60  0000 C CNN
-F 1 "74HC02" H 10850 1650 60  0000 C CNN
+F 1 "74HC02" H 10850 1650 60  0001 C CNN
 F 2 "" H 10800 1700 60  0000 C CNN
 F 3 "" H 10800 1700 60  0000 C CNN

Commit message: Added power pin units to most parts, +4VDC and +4VSW power components, and updated Scaler to use it all.
Parts:
- renumbered U1059 to U1159, U1060 to U1160, U1061 to U1161, U1062 to U1162
Changed lines of the file:
@@
 F33A
 $Comp
-L 74HC02 U1060
+L 74HC02 U1160
 U 1 1 56536164
 P 12950 1700
-F 0 "U1060" H 12950 1750 60  0000 C CNN
+F 0 "U1160" H 12950 1750 60  0000 C CNN
 F 1 "74HC02" H 13000 1650 60  0001 C CNN
 F 2 "" H 12950 1700 60  0000 C CNN
@@
 $EndComp
 $Comp
-L 74HC02 U1060
+L 74HC02 U1160
 U 2 1 5653616B
 P 15100 1700
-F 0 "U1060" H 15100 1750 60  0000 C CNN
+F 0 "U1160" H 15100 1750 60  0000 C CNN
 F 1 "74HC02" H 15150 1650 60  0001 C CNN
 F 2 "" H 15100 1700 60  0000 C CNN
@@
 $EndComp
 $Comp
-L 74HC02 U1060
+L 74HC02 U1160
 U 3 1 56536172
 P 17250 1700
-F 0 "U1060" H 17250 1750 60  0000 C CNN
+F 0 "U1160" H 17250 1750 60  0000 C CNN
 F 1 "74HC02" H 17300 1650 60  0001 C CNN
 F 2 "" H 17250 1700 60  0000 C CNN
@@
 $EndComp
 $Comp
-L 74HC02 U1060
+L 74HC02 U1160
 U 4 1 56536179
 P 19400 1700
-F 0 "U1060" H 19400 1750 60  0000 C CNN
+F 0 "U1160" H 19400 1750 60  0000 C CNN
 F 1 "74HC02" H 19450 1650 60  0001 C CNN
 F 2 "" H 19400 1700 60  0000 C CNN
@@
 	1950 4300 2100 4300
 $Comp
-L 74HC02 U1061
+L 74HC02 U1161
 U 1 1 56536184
 P 4350 3800
-F 0 "U1061" H 4350 3850 60  0000 C CNN
+F 0 "U1161" H 4350 3850 60  0000 C CNN
 F 1 "74HC02" H 4400 3750 60  0001 C CNN
 F 2 "" H 4350 3800 60  0000 C CNN
@@
 $EndComp
 $Comp
-L 74HC02 U1061
+L 74HC02 U1161
 U 2 1 5653618B
 P 6500 3800
-F 0 "U1061" H 6500 3850 60  0000 C CNN
+F 0 "U1161" H 6500 3850 60  0000 C CNN
 F 1 "74HC02" H 6550 3750 60  0001 C CNN
 F 2 "" H 6500 3800 60  0000 C CNN
@@
 $EndComp
 $Comp
-L 74HC02 U1061
+L 74HC02 U1161
 U 3 1 56536192
 P 8650 3800
-F 0 "U1061" H 8650 3850 60  0000 C CNN
+F 0 "U1161" H 8650 3850 60  0000 C CNN
 F 1 "74HC02" H 8700 3750 60  0001 C CNN
 F 2 "" H 8650 3800 60  0000 C CNN
@@
 $EndComp
 $Comp
-L 74HC02 U1061
+L 74HC02 U1161
 U 4 1 56536199
 P 10800 3800
-F 0 "U1061" H 10800 3850 60  0000 C CNN
+F 0 "U1161" H 10800 3850 60  0000 C CNN
 F 1 "74HC02" H 10850 3750 60  0001 C CNN
 F 2 "" H 10800 3800 60  0000 C CNN
@@
 $EndComp
 $Comp
-L 74HC02 U1062
+L 74HC02 U1162
 U 1 1 565361A0
 P 12950 3800
-F 0 "U1062" H 12950 3850 60  0000 C CNN
+F 0 "U1162" H 12950 3850 60  0000 C CNN
 F 1 "74HC02" H 13000 3750 60  0001 C CNN
 F 2 "" H 12950 3800 60  0000 C CNN
@@
 $EndComp
 $Comp
-L 74HC02 U1062
+L 74HC02 U1162
 U 2 1 565361A7
 P 15100 3800
-F 0 "U1062" H 15100 3850 60  0000 C CNN
+F 0 "U1162" H 15100 3850 60  0000 C CNN
 F 1 "74HC02" H 15150 3750 60  0001 C CNN
 F 2 "" H 15100 3800 60  0000 C CNN
@@
 $EndComp
 $Comp
-L 74HC02 U1062
+L 74HC02 U1162
 U 3 1 565361AE
 P 17250 3800
-F 0 "U1062" H 17250 3850 60  0000 C CNN
+F 0 "U1162" H 17250 3850 60  0000 C CNN
 F 1 "74HC02" H 17300 3750 60  0001 C CNN
 F 2 "" H 17250 3800 60  0000 C CNN
@@
 $EndComp
 $Comp
-L 74HC02 U1062
+L 74HC02 U1162
 U 4 1 565361B5
 P 19400 3800
-F 0 "U1062" H 19400 3850 60  0000 C CNN
+F 0 "U1162" H 19400 3850 60  0000 C CNN
 F 1 "74HC02" H 19450 3750 60  0001 C CNN
 F 2 "" H 19400 3800 60  0000 C CNN
@@
 Connection ~ 16650 3500
 $Comp
-L 74HC02 U1059
+L 74HC02 U1159
 U 1 1 5665597C
 P 4350 1700
-F 0 "U1059" H 4350 1750 60  0000 C CNN
+F 0 "U1159" H 4350 1750 60  0000 C CNN
 F 1 "74HC02" H 4400 1650 60  0001 C CNN
 F 2 "" H 4350 1700 60  0000 C CNN
@@
 $EndComp
 $Comp
-L 74HC02 U1059
+L 74HC02 U1159
 U 2 1 5666FE7D
 P 6500 1700
-F 0 "U1059" H 6500 1750 60  0000 C CNN
+F 0 "U1159" H 6500 1750 60  0000 C CNN
 F 1 "74HC02" H 6550 1650 60  0001 C CNN
 F 2 "" H 6500 1700 60  0000 C CNN
@@
 $EndComp
 $Comp
-L 74HC02 U1059
+L 74HC02 U1159
 U 3 1 5667E60A
 P 8650 1700
-F 0 "U1059" H 8650 1750 60  0000 C CNN
+F 0 "U1159" H 8650 1750 60  0000 C CNN
 F 1 "74HC02" H 8700 1650 60  0001 C CNN
 F 2 "" H 8650 1700 60  0000 C CNN
@@
 $EndComp
 $Comp
-L 74HC02 U1059
+L 74HC02 U1159
 U 4 1 56683D6C
 P 10800 1700
-F 0 "U1059" H 10800 1750 60  0000 C CNN
+F 0 "U1159" H 10800 1750 60  0000 C CNN
 F 1 "74HC02" H 10850 1650 60  0001 C CNN
 F 2 "" H 10800 1700 60  0000 C CNN
