File: four_bit_4/four_bit_4.sch (KiCad schematic (older format))
At the start: 1 part, among them P1 DIN_41612_128P

Commit message: Added interrupt inhibition to module 3
Connections:
- net EAC/: now also P1.65 (1C); no longer P1.63 (31B)
- net G13: now also P1.66 (2C); no longer P1.64 (32B)
- net G13/: now also P1.67 (3C); no longer P1.65 (1C)
- net G14: now also P1.68 (4C); no longer P1.66 (2C)
- net G14/: now also P1.69 (5C); no longer P1.67 (3C)
- net G15: now also P1.70 (6C); no longer P1.68 (4C)
- net G15/: now also P1.71 (7C); no longer P1.69 (5C)
- net G16: now also P1.72 (8C); no longer P1.70 (6C)
- net GEM13: now also P1.94 (30C); no longer P1.92 (28C)
- net GEM14: now also P1.95 (31C); no longer P1.93 (29C)
- net GEM16: now also P1.96 (32C); no longer P1.94 (30C)
- net GND: no longer P1.95 (31C), P1.96 (32C)
- net L15/: now also P1.73 (9C); no longer P1.71 (7C)
- net RL13/: now also P1.74 (10C); no longer P1.72 (8C)
- net RL14/: now also P1.75 (11C); no longer P1.73 (9C)
- net RL15/: now also P1.76 (12C); no longer P1.74 (10C)
- net RL16/: now also P1.77 (13C); no longer P1.75 (11C)
- net SUMA13/: now also P1.78 (14C); no longer P1.76 (12C)
- net SUMA14/: now also P1.80 (16C); no longer P1.78 (14C)
- net SUMA15/: now also P1.82 (18C); no longer P1.80 (16C)
- net SUMA16/: now also P1.84 (20C); no longer P1.82 (18C)
- net SUMB13/: now also P1.79 (15C); no longer P1.77 (13C)
- net SUMB14/: now also P1.81 (17C); no longer P1.79 (15C)
- net SUMB15/: now also P1.83 (19C); no longer P1.81 (17C)
- net SUMB16/: now also P1.85 (21C); no longer P1.83 (19C)
- net WL13/: now also P1.86 (22C); no longer P1.84 (20C)
- net WL14/: now also P1.87 (23C); no longer P1.85 (21C)
- net WL15: now also P1.88 (24C); no longer P1.86 (22C)
- net WL15/: now also P1.89 (25C); no longer P1.87 (23C)
- net WL16: now also P1.90 (26C); no longer P1.88 (24C)
- net WL16/: now also P1.91 (27C); no longer P1.89 (25C)
- net XUY13/: now also P1.92 (28C); no longer P1.90 (26C)
- net XUY14/: now also P1.93 (29C); no longer P1.91 (27C)
- new net A15/: P1.63 (31B)
- new net A16/: P1.64 (32B)
Changed lines of the file:
@@
 Text GLabel 4500 8350 0    60   Input ~ 0
 WL16/
-$Comp
-L GND #PWR07
-U 1 1 568CD535
-P 10250 4200
-F 0 "#PWR07" H 10250 3950 50  0001 C CNN
-F 1 "GND" H 10250 4050 50  0000 C CNN
-F 2 "" H 10250 4200 60  0000 C CNN
-F 3 "" H 10250 4200 60  0000 C CNN
-	1    10250 4200
-	1    0    0    -1
-$EndComp
 Text Label 6150 2000 0    60   ~ 0
 G16/
@@
 Wire Wire Line
 	4600 8350 4500 8350
-Wire Wire Line
-	10250 3950 10350 3950
-Wire Wire Line
-	10250 4050 10350 4050
-Connection ~ 10250 4050
 Wire Wire Line
 	6000 2000 6850 2000
@@
 Wire Wire Line
 	6000 1800 6100 1800
-Text GLabel 10250 950  0    60   Input ~ 0
+Text GLabel 10250 1150 0    60   Input ~ 0
 G13/
-Wire Wire Line
-	10350 950  10250 950
-Text GLabel 10250 1150 0    60   Input ~ 0
-G14/
 Wire Wire Line
 	10350 1150 10250 1150
 Text GLabel 10250 1350 0    60   Input ~ 0
+G14/
+Wire Wire Line
+	10350 1350 10250 1350
+Text GLabel 10250 1550 0    60   Input ~ 0
 G15/
 Wire Wire Line
-	10350 1350 10250 1350
+	10350 1550 10250 1550
 Text GLabel 6100 2100 2    60   Output ~ 0
 L15/
 Wire Wire Line
 	6000 2100 6100 2100
-Text GLabel 10250 1550 0    60   Input ~ 0
+Text GLabel 10250 1750 0    60   Input ~ 0
 L15/
 Wire Wire Line
-	10350 1550 10250 1550
+	10350 1750 10250 1750
 Text GLabel 6100 3050 2    60   Output ~ 0
 SUMA16/
@@
 Wire Wire Line
 	6000 3250 6100 3250
-Text GLabel 10250 2650 0    60   Input ~ 0
+Text GLabel 10250 2850 0    60   Input ~ 0
 SUMA16/
 Wire Wire Line
-	10350 2650 10250 2650
-Text GLabel 10250 2750 0    60   Input ~ 0
+	10350 2850 10250 2850
+Text GLabel 10250 2950 0    60   Input ~ 0
 SUMB16/
 Wire Wire Line
-	10350 2750 10250 2750
+	10350 2950 10250 2950
 Text GLabel 3250 3350 2    60   Output ~ 0
 XUY13/
@@
 Wire Wire Line
 	3150 3450 3250 3450
-Text GLabel 10250 3450 0    60   Input ~ 0
+Text GLabel 10250 3650 0    60   Input ~ 0
 XUY13/
 Wire Wire Line
-	10350 3450 10250 3450
-Text GLabel 10250 3550 0    60   Input ~ 0
+	10350 3650 10250 3650
+Text GLabel 10250 3750 0    60   Input ~ 0
 XUY14/
 Wire Wire Line
-	10350 3550 10250 3550
+	10350 3750 10250 3750
 Text GLabel 6100 4050 2    60   Output ~ 0
 WL15
@@
 Wire Wire Line
 	6000 4250 6100 4250
-Text GLabel 10250 2850 0    60   Input ~ 0
+Text GLabel 10250 3050 0    60   Input ~ 0
 WL13/
-Text GLabel 10250 2950 0    60   Input ~ 0
+Text GLabel 10250 3150 0    60   Input ~ 0
 WL14/
 Wire Wire Line
-	10350 2850 10250 2850
-Wire Wire Line
-	10350 2950 10250 2950
-Text GLabel 10250 3150 0    60   Input ~ 0
+	10350 3050 10250 3050
+Wire Wire Line
+	10350 3150 10250 3150
+Text GLabel 10250 3350 0    60   Input ~ 0
 WL15/
 Wire Wire Line
-	10350 3150 10250 3150
-Wire Wire Line
 	10350 3350 10250 3350
-Text GLabel 10250 3050 0    60   Input ~ 0
+Wire Wire Line
+	10350 3550 10250 3550
+Text GLabel 10250 3250 0    60   Input ~ 0
 WL15
-Text GLabel 10250 3250 0    60   Input ~ 0
+Text GLabel 10250 3450 0    60   Input ~ 0
 WL16
 Wire Wire Line
-	10350 3050 10250 3050
-Wire Wire Line
 	10350 3250 10250 3250
-Text GLabel 10250 3350 0    60   Input ~ 0
+Wire Wire Line
+	10350 3450 10250 3450
+Text GLabel 10250 3550 0    60   Input ~ 0
 WL16/
 Text GLabel 6100 2750 2    60   Output ~ 0
@@
 Wire Wire Line
 	6000 2750 6100 2750
-Text GLabel 9200 3950 0    60   Input ~ 0
+Text GLabel 10250 950  0    60   Input ~ 0
 EAC/
 Wire Wire Line
-	9300 3950 9200 3950
+	10350 950  10250 950
 Text GLabel 6100 2950 2    60   Output ~ 0
 SUMA15/
@@
 Wire Wire Line
 	6000 2950 6100 2950
-Text GLabel 10250 2450 0    60   Input ~ 0
+Text GLabel 10250 2650 0    60   Input ~ 0
 SUMA15/
 Wire Wire Line
-	10350 2450 10250 2450
-Text GLabel 10250 2550 0    60   Input ~ 0
+	10350 2650 10250 2650
+Text GLabel 10250 2750 0    60   Input ~ 0
 SUMB15/
 Wire Wire Line
-	10350 2550 10250 2550
+	10350 2750 10250 2750
 $Comp
 L GND #PWR014
@@
 Wire Wire Line
 	6000 1900 6100 1900
-Text GLabel 9200 4050 0    60   Input ~ 0
+Text GLabel 10250 1050 0    60   Input ~ 0
 G13
-Wire Wire Line
-	9300 4050 9200 4050
-Text GLabel 10250 1050 0    60   Input ~ 0
-G14
 Wire Wire Line
 	10350 1050 10250 1050
 Text GLabel 10250 1250 0    60   Input ~ 0
-G15
+G14
 Wire Wire Line
 	10350 1250 10250 1250
 Text GLabel 10250 1450 0    60   Input ~ 0
+G15
+Wire Wire Line
+	10350 1450 10250 1450
+Text GLabel 10250 1650 0    60   Input ~ 0
 G16
 Wire Wire Line
-	10350 1450 10250 1450
+	10350 1650 10250 1650
 Text GLabel 7350 2200 2    60   Input ~ 0
 L16/
@@
 Wire Wire Line
 	3150 3250 3250 3250
-Text GLabel 10250 2050 0    60   Input ~ 0
+Text GLabel 10250 2250 0    60   Input ~ 0
 SUMA13/
 Wire Wire Line
-	10350 2050 10250 2050
-Text GLabel 10250 2250 0    60   Input ~ 0
+	10350 2250 10250 2250
+Text GLabel 10250 2450 0    60   Input ~ 0
 SUMA14/
 Wire Wire Line
-	10350 2250 10250 2250
-Text GLabel 10250 2150 0    60   Input ~ 0
+	10350 2450 10250 2450
+Text GLabel 10250 2350 0    60   Input ~ 0
 SUMB13/
 Wire Wire Line
-	10350 2150 10250 2150
-Text GLabel 10250 2350 0    60   Input ~ 0
+	10350 2350 10250 2350
+Text GLabel 10250 2550 0    60   Input ~ 0
 SUMB14/
 Wire Wire Line
-	10350 2350 10250 2350
+	10350 2550 10250 2550
 Text GLabel 3250 3850 2    60   BiDi ~ 0
 RL13/
@@
 Wire Wire Line
 	6000 3950 6100 3950
-Text GLabel 10250 1650 0    60   BiDi ~ 0
+Text GLabel 10250 1850 0    60   BiDi ~ 0
 RL13/
-Wire Wire Line
-	10350 1650 10250 1650
-Text GLabel 10250 1750 0    60   BiDi ~ 0
-RL14/
-Wire Wire Line
-	10350 1750 10250 1750
-Text GLabel 10250 1850 0    60   BiDi ~ 0
-RL15/
 Wire Wire Line
 	10350 1850 10250 1850
 Text GLabel 10250 1950 0    60   BiDi ~ 0
+RL14/
+Wire Wire Line
+	10350 1950 10250 1950
+Text GLabel 10250 2050 0    60   BiDi ~ 0
+RL15/
+Wire Wire Line
+	10350 2050 10250 2050
+Text GLabel 10250 2150 0    60   BiDi ~ 0
 RL16/
 Wire Wire Line
-	10350 1950 10250 1950
+	10350 2150 10250 2150
 Text GLabel 3250 3600 2    60   Output ~ 0
 GEM13
@@
 Wire Wire Line
 	6000 3700 6100 3700
-Wire Wire Line
-	10250 3950 10250 4200
-Text GLabel 10250 3750 0    60   Input ~ 0
+Text GLabel 10250 3950 0    60   Input ~ 0
 GEM14
 Wire Wire Line
-	10350 3750 10250 3750
+	10350 3950 10250 3950
+Text GLabel 10250 4050 0    60   Input ~ 0
+GEM16
+Wire Wire Line
+	10350 4050 10250 4050
+Wire Wire Line
+	10350 3850 10250 3850
 Text GLabel 10250 3850 0    60   Input ~ 0
-GEM16
-Wire Wire Line
-	10350 3850 10250 3850
-Wire Wire Line
-	10350 3650 10250 3650
-Text GLabel 10250 3650 0    60   Input ~ 0
 GEM13
+Text GLabel 6100 1300 2    60   Output ~ 0
+A15/
+Wire Wire Line
+	6000 1300 6100 1300
+Text GLabel 6100 1400 2    60   Output ~ 0
+A16/
+Wire Wire Line
+	6000 1400 6100 1400
+Text GLabel 9200 4050 0    60   Input ~ 0
+A16/
+Wire Wire Line
+	9300 4050 9200 4050
+Text GLabel 9200 3950 0    60   Input ~ 0
+A15/
+Wire Wire Line
+	9300 3950 9200 3950
 $EndSCHEMATC

Commit message: Added and tied in Inout VII, the final logic module!
I still need to comb through the schematics to see if there are any
stray gates I missed. The initial conditions are also pretty much
guaranteed to be wrong. But it's mostly all there!
Connections:
- net GEM13: now also P1.96 (32C); no longer P1.94 (30C)
- net GEM14: now also P1.97 (1D); no longer P1.95 (31C)
- net GEM16: now also P1.98 (2D); no longer P1.96 (32C)
- net GND: no longer P1.97 (1D), P1.98 (2D)
- net WL13/: now also P1.87 (23C); no longer P1.86 (22C)
- net WL14/: now also P1.89 (25C); no longer P1.87 (23C)
- net WL15: now also P1.90 (26C); no longer P1.88 (24C)
- net WL15/: now also P1.91 (27C); no longer P1.89 (25C)
- net WL16: now also P1.92 (28C); no longer P1.90 (26C)
- net WL16/: now also P1.93 (29C); no longer P1.91 (27C)
- net XUY13/: now also P1.94 (30C); no longer P1.92 (28C)
- net XUY14/: now also P1.95 (31C); no longer P1.93 (29C)
- new net WL13: P1.86 (22C)
- new net WL14: P1.88 (24C)
Changed lines of the file:
@@
 L13/
 Wire Wire Line
-	11500 950  11400 950
-Wire Wire Line
-	11500 1050 11400 1050
-Connection ~ 11400 1050
-Wire Wire Line
 	11400 1150 11500 1150
-Connection ~ 11400 1150
 Wire Wire Line
 	11400 1250 11500 1250
@@
 	11400 4050 11500 4050
 Connection ~ 11400 4050
-Wire Wire Line
-	11400 950  11400 4200
 Wire Wire Line
 	12300 950  12200 950
@@
 Wire Wire Line
 	3150 3450 3250 3450
-Text GLabel 10250 3650 0    60   Input ~ 0
+Text GLabel 10250 3850 0    60   Input ~ 0
 XUY13/
 Wire Wire Line
-	10350 3650 10250 3650
-Text GLabel 10250 3750 0    60   Input ~ 0
+	10350 3850 10250 3850
+Text GLabel 10250 3950 0    60   Input ~ 0
 XUY14/
 Wire Wire Line
-	10350 3750 10250 3750
+	10350 3950 10250 3950
 Text GLabel 6100 4050 2    60   Output ~ 0
 WL15
@@
 Wire Wire Line
 	6000 4250 6100 4250
-Text GLabel 10250 3050 0    60   Input ~ 0
+Text GLabel 10250 3150 0    60   Input ~ 0
 WL13/
-Text GLabel 10250 3150 0    60   Input ~ 0
+Text GLabel 10250 3350 0    60   Input ~ 0
 WL14/
 Wire Wire Line
-	10350 3050 10250 3050
-Wire Wire Line
 	10350 3150 10250 3150
-Text GLabel 10250 3350 0    60   Input ~ 0
+Wire Wire Line
+	10350 3350 10250 3350
+Text GLabel 10250 3550 0    60   Input ~ 0
 WL15/
 Wire Wire Line
-	10350 3350 10250 3350
-Wire Wire Line
 	10350 3550 10250 3550
-Text GLabel 10250 3250 0    60   Input ~ 0
+Wire Wire Line
+	10350 3750 10250 3750
+Text GLabel 10250 3450 0    60   Input ~ 0
 WL15
-Text GLabel 10250 3450 0    60   Input ~ 0
+Text GLabel 10250 3650 0    60   Input ~ 0
 WL16
 Wire Wire Line
-	10350 3250 10250 3250
-Wire Wire Line
 	10350 3450 10250 3450
-Text GLabel 10250 3550 0    60   Input ~ 0
+Wire Wire Line
+	10350 3650 10250 3650
+Text GLabel 10250 3750 0    60   Input ~ 0
 WL16/
 Text GLabel 6100 2750 2    60   Output ~ 0
@@
 Wire Wire Line
 	6000 3700 6100 3700
-Text GLabel 10250 3950 0    60   Input ~ 0
+Text GLabel 11400 950  0    60   Input ~ 0
 GEM14
 Wire Wire Line
-	10350 3950 10250 3950
+	11500 950  11400 950
+Text GLabel 11400 1050 0    60   Input ~ 0
+GEM16
+Wire Wire Line
+	11500 1050 11400 1050
+Wire Wire Line
+	10350 4050 10250 4050
 Text GLabel 10250 4050 0    60   Input ~ 0
-GEM16
-Wire Wire Line
-	10350 4050 10250 4050
-Wire Wire Line
-	10350 3850 10250 3850
-Text GLabel 10250 3850 0    60   Input ~ 0
 GEM13
 Text GLabel 6100 1300 2    60   Output ~ 0
@@
 Wire Wire Line
 	9300 3950 9200 3950
+Text GLabel 3250 4050 2    60   Output ~ 0
+WL13
+Text GLabel 3250 4250 2    60   Output ~ 0
+WL14
+Wire Wire Line
+	3150 4050 3250 4050
+Wire Wire Line
+	3150 4250 3250 4250
+Wire Wire Line
+	11400 1150 11400 4200
+Text GLabel 10250 3050 0    60   Input ~ 0
+WL13
+Text GLabel 10250 3250 0    60   Input ~ 0
+WL14
+Wire Wire Line
+	10350 3050 10250 3050
+Wire Wire Line
+	10350 3250 10250 3250
 $EndSCHEMATC
