File: service_gates/a07_2.sch (KiCad schematic (older format))
At the start: 25 parts, among them U7016 74HC04, U7018 74HC02, U7019 74HC27, U7020 74HC02, U7021 74HC02, U7022 74HC04, U7023 74HC02, U7024 74HC27, U7025 74HC02, U7026 74HC04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

Commit message: Tied in module 7, and corrected lots of errors.
Off the top of my head:
* T12DC/ not actually connected to restart logic in A02-2
* IC12/ and IC13 schematic errors
* Lots of gates moved from later modules up to modules 2-7
* YT0..7 logic dropped from 7, it belongs in 14
* Lots of missing signal breakouts
* ...probably some other things, I should keep a list as I go

All control pulses associated with GOJ1 now behave correctly during
GOJ1.
Parts:
- removed unit 3 of U7029
- removed unit 6 of U7031
- removed U7033, U7035: 74HC04, symbol 74HC04
- removed U7034, U7036: 74HC27, symbol 74HC27
- removed unit 1 of U7037
- removed unit 2 of U7037
- removed unit 3 of U7037
- removed unit 1 of U7038
- added unit 6 of U7041
Connections:
- net GND: now also U7041.7 (GND)
- net U2BBK: now also U7041.13
- net VCC: now also U7041.14 (VCC)
- new net U2BBKG/: U7041.12
Other:
- note removed: "Of all of these outputs, only YT0/ is used. Good candidates for removal."
- moved on the sheet: U7037D, U7038B, U7039A, U7039B, U7039C

Commit message: Tied in module 8, and corrected lots of initial conditions.
The registers and ALU appear to work now, with TC0 and STD2 shuffling things around correctly, and Z counting up as instructions execute.
Parts:
- U7016, U7022: Initial (none) -> 1
Changed lines of the file:
@@
 F 2 "" H 3400 4450 60  0000 C CNN
 F 3 "" H 3400 4450 60  0000 C CNN
+F 4 "1" H 3450 4450 60  0000 C CIN "Initial"
 	6    3400 4450
 	1    0    0    -1
@@
 F 2 "" H 3400 5350 60  0000 C CNN
 F 3 "" H 3400 5350 60  0000 C CNN
+F 4 "1" H 3450 5350 60  0000 C CIN "Initial"
 	2    3400 5350
 	1    0    0    -1

Commit message: Added the final four bit module. All 16 bits of the central/special registers are present. We're stuck at address 0 because TC is using RAD, which needs to be translated into RG or RZ by module 12
Parts:
- added unit 3 of U7029
Connections:
- net GND: now also U7029.7 (GND)
- net RUSG/: now also U7029.9
- net VCC: now also U7029.14 (VCC)
- new net SUMA15/: U7029.10
- new net SUMB15/: U7029.11
- new net US2SG: U7029.8
Changed lines of the file:
@@
 MRULOG
 Wire Wire Line
-	10700 6450 11850 6450
-Text HLabel 11850 6450 2    60   Output ~ 0
-RUSG/
+	10700 6450 11150 6450
+Text HLabel 12500 6600 2    60   Output ~ 0
+US2SG
 $Comp
 L 74HC02 U7032
@@
 Text HLabel 2450 9850 2    60   Output ~ 0
 U2BBKG/
+Text Label 10700 6450 0    60   ~ 0
+RUSG/
+$Comp
+L 74HC27 U7029
+U 3 1 56B1B183
+P 11750 6600
+F 0 "U7029" H 11750 6650 60  0000 C CNN
+F 1 "74HC27" H 11750 6550 60  0000 C CNN
+F 2 "" H 11750 6600 60  0000 C CNN
+F 3 "" H 11750 6600 60  0000 C CNN
+	3    11750 6600
+	1    0    0    -1
+$EndComp
+Wire Wire Line
+	12500 6600 12350 6600
+Text HLabel 11050 6600 0    60   Input ~ 0
+SUMA15/
+Wire Wire Line
+	11050 6600 11150 6600
+Text HLabel 11050 6750 0    60   Input ~ 0
+SUMB15/
+Wire Wire Line
+	11050 6750 11150 6750
 $EndSCHEMATC

Commit message: Added and tied in module 12, parity & s register
Parts:
- U7022: Initial (none) -> 1
Changed lines of the file:
@@
 F 2 "" H 3400 4850 60  0000 C CNN
 F 3 "" H 3400 4850 60  0000 C CNN
+F 4 "1" H 3400 4850 60  0000 C CIN "Initial"
 	1    3400 4850
 	1    0    0    -1

Commit message: Added and tied in module 15, the rupt service (and banking/rope+strand selection)
Parts:
- added unit 1 of U7037
- U7022, U7025, U7041: Initial (none) -> 1
Connections:
- net GND: now also U7037.7 (GND)
- net VCC: now also U7037.14 (VCC)
- net WEBG/: now also U7037.2; no longer U7023.10, U7024.3
- new net: U7023.10, U7024.3, U7037.1
Other:
- moved on the sheet: U7022D, U7022E, U7022F, U7023D, U7024B, U7024C, U7025A, U7025B, U7025C, U7025D, U7026A, U7041F

Commit message: Added erasable memory, and fixed lots of random wiring errors.
I decided to go with a 16-bit-wide MRAM chip -- I had  no idea
until I started researching RAM options how technologically
similar MRAM is to core memory. The datasheet diagrams look like
they're straight out of the AGC documentation!

There's a slight inaccuracy in this implementation worth mentioning.
Like fixed memory, I've wired the sense amplifier outputs directly up
to the tristate data output pins of the MRAM chip. But because the
data lines are bidirectional, data being written into RAM will show up
on the sense lines, and go straight into the ungated G register. Since
G is what's being written out, this doesn't matter 99% of the time, but
if there's an overflow condition in G (I don't even know if this is
possible), the bit 16 will be copied over bit 16, and the overflow
condition will be lost. I'll keep an eye out to see if anything relies
on G not changing after the write cycle is complete.

With erasable memory introduced, the computer now theoretically supports
all programs that don't use I/O or interrupts. I've started running
the VirtualAGC validation program, and have been fixing random errors
uncovered by failing self-tests.
Connections:
- net T10/: no longer U7025.6
- net XB4/: now also U7025.6
Changed lines of the file:
@@
 	1450 9650 1100 9650
-Wire Wire Line
-	1200 3150 1200 9050
-Connection ~ 1200 3150
 Wire Wire Line
 	1200 9050 1450 9050
@@
 	3900 6900 3900 7100
 Connection ~ 3900 7100
+Wire Wire Line
+	1200 2850 1200 9050
+Connection ~ 1200 2850
 $EndSCHEMATC

Commit message: Not gate rewiring up through module 11, with other cleanup here and there
Parts:
- U7039: Initial (none) -> 1
Other:
- moved on the sheet: U7016E, U7016F, U7021B, U7021C, U7022A, U7022B, U7022C, U7022D, U7022E, U7022F, U7023A, U7023B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
