File: dsky/indicator_driver/line_driver.sch (KiCad schematic (older format))
At the start: 12 parts, among them Q7 PN2222AA, Q8 PN2222AA

Commit message: Finished initial wiring of the Indicator Driver Module. Currently sitting at 111 pins used, so I've been too aggressive at culling pins
Changed lines of the file:
@@
 Wire Wire Line
 	5000 2000 5450 2000
-Text HLabel 5450 2000 2    60   Input ~ 0
+Text HLabel 5450 2000 2    60   Output ~ 0
 RELAY_LINE
 $EndSCHEMATC

Commit message: DSKY IDM: Cleaned up design rule errors. Still don't fully understand the common returh path.
Changed lines of the file:
@@
 $Descr A4 11693 8268
 encoding utf-8
-Sheet 10 12
+Sheet 9 12
 Title ""
 Date ""
@@
 AR Path="/582AE841/582B1340" Ref="D81"  Part="1"
 AR Path="/582C01D3/582B1340" Ref="D85"  Part="1"
-F 0 "D85" H 3200 2300 50  0000 C CNN
+F 0 "D81" H 3200 2300 50  0000 C CNN
 F 1 "1N4148" H 3200 2100 50  0000 C CNN
 F 2 "" H 3200 2200 60  0000 C CNN
@@
 AR Path="/582AE841/582B1403" Ref="D82"  Part="1"
 AR Path="/582C01D3/582B1403" Ref="D86"  Part="1"
-F 0 "D86" H 3200 2650 50  0000 C CNN
+F 0 "D82" H 3200 2650 50  0000 C CNN
 F 1 "1N4148" H 3200 2450 50  0000 C CNN
 F 2 "" H 3200 2550 60  0000 C CNN
@@
 AR Path="/582AE841/582B141D" Ref="D83"  Part="1"
 AR Path="/582C01D3/582B141D" Ref="D87"  Part="1"
-F 0 "D87" H 3200 3000 50  0000 C CNN
+F 0 "D83" H 3200 3000 50  0000 C CNN
 F 1 "1N4148" H 3200 2800 50  0000 C CNN
 F 2 "" H 3200 2900 60  0000 C CNN
@@
 AR Path="/582AE841/582B1438" Ref="D84"  Part="1"
 AR Path="/582C01D3/582B1438" Ref="D88"  Part="1"
-F 0 "D88" H 3200 3350 50  0000 C CNN
+F 0 "D84" H 3200 3350 50  0000 C CNN
 F 1 "1N4148" H 3200 3150 50  0000 C CNN
 F 2 "" H 3200 3250 60  0000 C CNN
@@
 AR Path="/582AE841/582B14F9" Ref="R10"  Part="1"
 AR Path="/582C01D3/582B14F9" Ref="R16"  Part="1"
-F 0 "R16" V 2980 3600 50  0000 C CNN
+F 0 "R10" V 2980 3600 50  0000 C CNN
 F 1 "1k" V 2900 3600 50  0000 C CNN
 F 2 "" V 2830 3600 30  0000 C CNN
@@
 AR Path="/582AE841/582B1AC1" Ref="R11"  Part="1"
 AR Path="/582C01D3/582B1AC1" Ref="R17"  Part="1"
-F 0 "R17" V 2780 3600 50  0000 C CNN
+F 0 "R11" V 2780 3600 50  0000 C CNN
 F 1 "1k" V 2700 3600 50  0000 C CNN
 F 2 "" V 2630 3600 30  0000 C CNN
@@
 AR Path="/582AE841/582B1B16" Ref="R12"  Part="1"
 AR Path="/582C01D3/582B1B16" Ref="R18"  Part="1"
-F 0 "R18" V 2580 3600 50  0000 C CNN
+F 0 "R12" V 2580 3600 50  0000 C CNN
 F 1 "1k" V 2500 3600 50  0000 C CNN
 F 2 "" V 2430 3600 30  0000 C CNN
@@
 AR Path="/582AE841/582B1B1C" Ref="R13"  Part="1"
 AR Path="/582C01D3/582B1B1C" Ref="R19"  Part="1"
-F 0 "R19" V 2380 3600 50  0000 C CNN
+F 0 "R13" V 2380 3600 50  0000 C CNN
 F 1 "1k" V 2300 3600 50  0000 C CNN
 F 2 "" V 2230 3600 30  0000 C CNN
@@
 Connection ~ 2700 3850
 $Comp
-L GND #PWR04
+L GND #PWR010
 U 1 1 582B1BA1
 P 2600 3950
-AR Path="/582AE841/582B1BA1" Ref="#PWR04"  Part="1"
-AR Path="/582C01D3/582B1BA1" Ref="#PWR07"  Part="1"
-F 0 "#PWR07" H 2600 3700 50  0001 C CNN
+AR Path="/582AE841/582B1BA1" Ref="#PWR010"  Part="1"
+AR Path="/582C01D3/582B1BA1" Ref="#PWR013"  Part="1"
+F 0 "#PWR013" H 2600 3700 50  0001 C CNN
 F 1 "GND" H 2600 3800 50  0000 C CNN
 F 2 "" H 2600 3950 60  0000 C CNN
@@
 AR Path="/582AE841/582B2579" Ref="R14"  Part="1"
 AR Path="/582C01D3/582B2579" Ref="R20"  Part="1"
-F 0 "R20" V 3580 2000 50  0000 C CNN
+F 0 "R14" V 3580 2000 50  0000 C CNN
 F 1 "100k" V 3500 2000 50  0000 C CNN
 F 2 "" V 3430 2000 30  0000 C CNN
@@
 $EndComp
 $Comp
-L +12V #PWR05
+L +12V #PWR011
 U 1 1 582B258A
 P 3500 1850
-AR Path="/582AE841/582B258A" Ref="#PWR05"  Part="1"
-AR Path="/582C01D3/582B258A" Ref="#PWR08"  Part="1"
-F 0 "#PWR08" H 3500 1700 50  0001 C CNN
+AR Path="/582AE841/582B258A" Ref="#PWR011"  Part="1"
+AR Path="/582C01D3/582B258A" Ref="#PWR014"  Part="1"
+F 0 "#PWR014" H 3500 1700 50  0001 C CNN
 F 1 "+12V" H 3500 1990 50  0000 C CNN
 F 2 "" H 3500 1850 60  0000 C CNN
@@
 AR Path="/582AE841/582B2973" Ref="Q7"  Part="1"
 AR Path="/582C01D3/582B2973" Ref="Q9"  Part="1"
-F 0 "Q9" H 4500 2600 50  0000 R CNN
+F 0 "Q7" H 4500 2600 50  0000 R CNN
 F 1 "PN2222AA" H 4750 2500 50  0000 R CNN
 F 2 "" H 4400 2650 29  0000 C CNN
@@
 AR Path="/582AE841/582B2AA5" Ref="Q8"  Part="1"
 AR Path="/582C01D3/582B2AA5" Ref="Q10"  Part="1"
-F 0 "Q10" H 5200 3000 50  0000 R CNN
+F 0 "Q8" H 5200 3000 50  0000 R CNN
 F 1 "PN2222AA" H 5450 2900 50  0000 R CNN
 F 2 "" H 5100 3050 29  0000 C CNN
@@
 $EndComp
 $Comp
-L GND #PWR06
+L GND #PWR012
 U 1 1 582B2C0D
 P 5000 3450
-AR Path="/582AE841/582B2C0D" Ref="#PWR06"  Part="1"
-AR Path="/582C01D3/582B2C0D" Ref="#PWR09"  Part="1"
-F 0 "#PWR09" H 5000 3200 50  0001 C CNN
+AR Path="/582AE841/582B2C0D" Ref="#PWR012"  Part="1"
+AR Path="/582C01D3/582B2C0D" Ref="#PWR015"  Part="1"
+F 0 "#PWR015" H 5000 3200 50  0001 C CNN
 F 1 "GND" H 5000 3300 50  0000 C CNN
 F 2 "" H 5000 3450 60  0000 C CNN
@@
 AR Path="/582AE841/582B2CB4" Ref="R15"  Part="1"
 AR Path="/582C01D3/582B2CB4" Ref="R21"  Part="1"
-F 0 "R21" V 4680 3150 50  0000 C CNN
+F 0 "R15" V 4680 3150 50  0000 C CNN
 F 1 "5k" V 4600 3150 50  0000 C CNN
 F 2 "" V 4530 3150 30  0000 C CNN
