File: dsky/indicator_driver/indicator_driver.sch (KiCad schematic (older format))
At the start: 1 part, among them P1 DIN_41612_128P

Commit message: DSKY IDM: Cleaned up design rule errors. Still don't fully understand the common returh path.
Connections:
- wire segments 141 -> 157
Changed lines of the file:
@@
 Comment4 ""
 $EndDescr
-$Sheet
-S 1350 3000 1250 1950
-U 57369BCB
-F0 "Decoder 1" 60
-F1 "seven_segment_decoder.sch" 60
-F2 "+250VAC" I L 1350 3100 60
-F3 "SEG_A" O R 2600 3100 60
-F4 "SEG_B" O R 2600 3200 60
-F5 "SEG_D" O R 2600 3400 60
-F6 "SEG_G" O R 2600 3700 60
-F7 "SEG_F" O R 2600 3600 60
-F8 "SEG_C" O R 2600 3300 60
-F9 "SEG_E" O R 2600 3500 60
-F10 "R5_SET" I L 1350 4600 60
-F11 "R5_RESET" I L 1350 4700 60
-F12 "R4_SET" I L 1350 4350 60
-F13 "R4_RESET" I L 1350 4450 60
-F14 "R3_SET" I L 1350 4100 60
-F15 "R3_RESET" I L 1350 4200 60
-F16 "R2_SET" I L 1350 3850 60
-F17 "R2_RESET" I L 1350 3950 60
-F18 "R1_SET" I L 1350 3600 60
-F19 "R1_RESET" I L 1350 3700 60
-F20 "R145_LINE/" I L 1350 3250 60
-F21 "R2_OUT" O R 2600 4850 60
-F22 "R15_IN" I L 1350 4850 60
-F23 "R2_LINE/" I L 1350 3350 60
-F24 "R3_LINE/" I L 1350 3450 60
-$EndSheet
 Wire Wire Line
 	2600 4850 2900 4850
@@
 $EndSheet
 $Sheet
-S 7150 5550 1050 700
+S 7000 4650 1050 700
 U 582E87BD
 F0 "Non-Latching Relay 1" 60
 F1 "nonlatching_relay.sch" 60
-F2 "RELAY_SET" I L 7150 5650 60
-F3 "C1" O R 8200 5850 60
-F4 "C2" O R 8200 6100 60
-F5 "NC1" I L 7150 5800 60
-F6 "NO1" I L 7150 5900 60
-F7 "NC2" I L 7150 6050 60
-F8 "NO2" I L 7150 6150 60
+F2 "RELAY_SET" I L 7000 4750 60
+F3 "C1" O R 8050 4950 60
+F4 "C2" O R 8050 5200 60
+F5 "NC1" I L 7000 4900 60
+F6 "NO1" I L 7000 5000 60
+F7 "NC2" I L 7000 5150 60
+F8 "NO2" I L 7000 5250 60
 $EndSheet
 Wire Wire Line
@@
 Relay Drivers
 $Sheet
-S 9400 5550 1050 700
+S 7000 5650 1050 700
 U 582FE107
 F0 "Non-Latching Relay 2" 60
 F1 "nonlatching_relay.sch" 60
-F2 "RELAY_SET" I L 9400 5650 60
-F3 "C1" O R 10450 5850 60
-F4 "C2" O R 10450 6100 60
-F5 "NC1" I L 9400 5800 60
-F6 "NO1" I L 9400 5900 60
-F7 "NC2" I L 9400 6050 60
-F8 "NO2" I L 9400 6150 60
+F2 "RELAY_SET" I L 7000 5750 60
+F3 "C1" O R 8050 5950 60
+F4 "C2" O R 8050 6200 60
+F5 "NC1" I L 7000 5900 60
+F6 "NO1" I L 7000 6000 60
+F7 "NC2" I L 7000 6150 60
+F8 "NO2" I L 7000 6250 60
 $EndSheet
 Wire Wire Line
-	7150 5650 7050 5650
-Text GLabel 7050 5650 0    60   Input ~ 0
+	7000 4750 6900 4750
+Text GLabel 6900 4750 0    60   Input ~ 0
 R21_S
 Wire Wire Line
-	7150 5800 7050 5800
-Text GLabel 7050 5800 0    60   Input ~ 0
+	7000 4900 6900 4900
+Text GLabel 6900 4900 0    60   Input ~ 0
 R21_NC1
 Wire Wire Line
-	7150 5900 7050 5900
-Text GLabel 7050 5900 0    60   Input ~ 0
+	7000 5000 6900 5000
+Text GLabel 6900 5000 0    60   Input ~ 0
 R21_NO1
 Wire Wire Line
-	7150 6050 7050 6050
-Text GLabel 7050 6050 0    60   Input ~ 0
+	7000 5150 6900 5150
+Text GLabel 6900 5150 0    60   Input ~ 0
 R21_NC2
 Wire Wire Line
-	7150 6150 7050 6150
-Text GLabel 7050 6150 0    60   Input ~ 0
+	7000 5250 6900 5250
+Text GLabel 6900 5250 0    60   Input ~ 0
 R21_NO2
 Wire Wire Line
-	8200 5850 8300 5850
-Text GLabel 8300 5850 2    60   Output ~ 0
+	8050 4950 8150 4950
+Text GLabel 8150 4950 2    60   Output ~ 0
 R21_C1
-Text GLabel 8300 6100 2    60   Output ~ 0
+Text GLabel 8150 5200 2    60   Output ~ 0
 R21_C2
 Wire Wire Line
-	8300 6100 8200 6100
-Wire Wire Line
-	9400 5650 9300 5650
-Text GLabel 9300 5650 0    60   Input ~ 0
+	8150 5200 8050 5200
+Wire Wire Line
+	7000 5750 6900 5750
+Text GLabel 6900 5750 0    60   Input ~ 0
 R22_S
 Wire Wire Line
-	9400 5800 9300 5800
-Text GLabel 9300 5800 0    60   Input ~ 0
+	7000 5900 6900 5900
+Text GLabel 6900 5900 0    60   Input ~ 0
 R22_NC1
 Wire Wire Line
-	9400 5900 9300 5900
-Text GLabel 9300 5900 0    60   Input ~ 0
+	7000 6000 6900 6000
+Text GLabel 6900 6000 0    60   Input ~ 0
 R22_NO1
 Wire Wire Line
-	9400 6050 9300 6050
-Text GLabel 9300 6050 0    60   Input ~ 0
+	7000 6150 6900 6150
+Text GLabel 6900 6150 0    60   Input ~ 0
 R22_NC2
 Wire Wire Line
-	9400 6150 9300 6150
-Text GLabel 9300 6150 0    60   Input ~ 0
+	7000 6250 6900 6250
+Text GLabel 6900 6250 0    60   Input ~ 0
 R22_NO2
-Text GLabel 10750 2250 0    60   UnSpc ~ 0
+Text GLabel 10750 2650 0    60   UnSpc ~ 0
 R22_C1
-Text GLabel 10750 2350 0    60   UnSpc ~ 0
+Text GLabel 10750 2750 0    60   UnSpc ~ 0
 R22_C2
 Wire Wire Line
-	10550 5850 10450 5850
-Wire Wire Line
-	10550 6100 10450 6100
+	8150 5950 8050 5950
+Wire Wire Line
+	8150 6200 8050 6200
 $Comp
 L DIN_41612_128P P1
@@
 Text GLabel 7450 2850 0    60   Input ~ 0
 RELAY_LINE_2
-Text GLabel 10750 1150 0    60   Output ~ 0
-+250VAC
 Wire Wire Line
 	10750 1050 10650 1050
 Wire Wire Line
-	10650 1050 10650 950
+	10650 950  10650 1350
 $Comp
-L +12V #PWR?
+L +12V #PWR01
 U 1 1 585336C8
 P 10650 950
-F 0 "#PWR?" H 10650 800 50  0001 C CNN
+F 0 "#PWR01" H 10650 800 50  0001 C CNN
 F 1 "+12V" H 10650 1090 50  0000 C CNN
 F 2 "" H 10650 950 60  0000 C CNN
@@
 	10750 4150 10650 4150
 Wire Wire Line
-	10650 4150 10650 4250
+	10650 2850 10650 4250
 $Comp
-L GND #PWR?
+L GND #PWR02
 U 1 1 585355DD
 P 10650 4250
-F 0 "#PWR?" H 10650 4000 50  0001 C CNN
+F 0 "#PWR02" H 10650 4000 50  0001 C CNN
 F 1 "GND" H 10650 4100 50  0000 C CNN
 F 2 "" H 10650 4250 60  0000 C CNN
@@
 Text GLabel 9800 4150 0    60   UnSpc ~ 0
 R21_NC1
-Text GLabel 10750 1250 0    60   UnSpc ~ 0
+Text GLabel 10750 1650 0    60   UnSpc ~ 0
 R21_NO1
-Text GLabel 10750 1350 0    60   UnSpc ~ 0
+Text GLabel 10750 1750 0    60   UnSpc ~ 0
 R21_NC2
-Text GLabel 10750 1450 0    60   UnSpc ~ 0
+Text GLabel 10750 1850 0    60   UnSpc ~ 0
 R21_NO2
-Text GLabel 10750 1750 0    60   Output ~ 0
+Text GLabel 10750 2150 0    60   Output ~ 0
 R22_S
-Text GLabel 10750 1850 0    60   UnSpc ~ 0
+Text GLabel 10750 2250 0    60   UnSpc ~ 0
 R22_NC1
+Text GLabel 10750 2350 0    60   UnSpc ~ 0
+R22_NO1
+Text GLabel 10750 2450 0    60   UnSpc ~ 0
+R22_NC2
+Text GLabel 10750 2550 0    60   UnSpc ~ 0
+R22_NO2
 Text GLabel 10750 1950 0    60   UnSpc ~ 0
-R22_NO1
+R21_C1
 Text GLabel 10750 2050 0    60   UnSpc ~ 0
-R22_NC2
-Text GLabel 10750 2150 0    60   UnSpc ~ 0
-R22_NO2
-Text GLabel 10750 1550 0    60   UnSpc ~ 0
-R21_C1
-Text GLabel 10750 1650 0    60   UnSpc ~ 0
 R21_C2
 Wire Wire Line
@@
 Text GLabel 9800 2050 0    60   Input ~ 0
 DEC4_LINE3/
-Text GLabel 10550 5850 2    60   Output ~ 0
+Text GLabel 8150 5950 2    60   Output ~ 0
 R22_C1
-Text GLabel 10550 6100 2    60   Output ~ 0
+Text GLabel 8150 6200 2    60   Output ~ 0
 R22_C2
+$Sheet
+S 1350 3000 1250 1950
+U 57369BCB
+F0 "Decoder 1" 60
+F1 "seven_segment_decoder.sch" 60
+F2 "+250VAC" I L 1350 3100 60
+F3 "SEG_A" O R 2600 3100 60
+F4 "SEG_B" O R 2600 3200 60
+F5 "SEG_D" O R 2600 3400 60
+F6 "SEG_G" O R 2600 3700 60
+F7 "SEG_F" O R 2600 3600 60
+F8 "SEG_C" O R 2600 3300 60
+F9 "SEG_E" O R 2600 3500 60
+F10 "R5_SET" I L 1350 4600 60
+F11 "R5_RESET" I L 1350 4700 60
+F12 "R4_SET" I L 1350 4350 60
+F13 "R4_RESET" I L 1350 4450 60
+F14 "R3_SET" I L 1350 4100 60
+F15 "R3_RESET" I L 1350 4200 60
+F16 "R2_SET" I L 1350 3850 60
+F17 "R2_RESET" I L 1350 3950 60
+F18 "R1_SET" I L 1350 3600 60
+F19 "R1_RESET" I L 1350 3700 60
+F20 "R145_LINE/" I L 1350 3250 60
+F21 "R2_OUT" O R 2600 4850 60
+F22 "R15_IN" I L 1350 4850 60
+F23 "R2_LINE/" I L 1350 3350 60
+F24 "R3_LINE/" I L 1350 3450 60
+$EndSheet
+Wire Wire Line
+	10650 4050 10750 4050
+Connection ~ 10650 4150
+Wire Wire Line
+	10650 3950 10750 3950
+Connection ~ 10650 4050
+Wire Wire Line
+	10650 3850 10750 3850
+Connection ~ 10650 3950
+Wire Wire Line
+	10650 3750 10750 3750
+Connection ~ 10650 3850
+Wire Wire Line
+	10650 3650 10750 3650
+Connection ~ 10650 3750
+Wire Wire Line
+	10650 3550 10750 3550
+Connection ~ 10650 3650
+Wire Wire Line
+	10650 3450 10750 3450
+Connection ~ 10650 3550
+Wire Wire Line
+	10650 3350 10750 3350
+Connection ~ 10650 3450
+Wire Wire Line
+	10650 3250 10750 3250
+Connection ~ 10650 3350
+Wire Wire Line
+	10650 3150 10750 3150
+Connection ~ 10650 3250
+Wire Wire Line
+	10650 3050 10750 3050
+Connection ~ 10650 3150
+Wire Wire Line
+	10650 2950 10750 2950
+Connection ~ 10650 3050
+Wire Wire Line
+	10650 1150 10750 1150
+Connection ~ 10650 1050
+Wire Wire Line
+	10650 1250 10750 1250
+Connection ~ 10650 1150
+Text GLabel 10750 1550 0    60   Output ~ 0
++250VAC
+Wire Wire Line
+	10750 2850 10650 2850
+Connection ~ 10650 2950
+$Comp
+L PWR_FLAG #FLG03
+U 1 1 586BAFD1
+P 11000 4750
+F 0 "#FLG03" H 11000 4845 50  0001 C CNN
+F 1 "PWR_FLAG" H 11000 4930 50  0000 C CNN
+F 2 "" H 11000 4750 60  0000 C CNN
+F 3 "" H 11000 4750 60  0000 C CNN
+	1    11000 4750
+	1    0    0    -1
+$EndComp
+$Comp
+L GND #PWR04
+U 1 1 586BB918
+P 11000 4750
+F 0 "#PWR04" H 11000 4500 50  0001 C CNN
+F 1 "GND" H 11000 4600 50  0000 C CNN
+F 2 "" H 11000 4750 60  0000 C CNN
+F 3 "" H 11000 4750 60  0000 C CNN
+	1    11000 4750
+	1    0    0    -1
+$EndComp
+$Comp
+L PWR_FLAG #FLG05
+U 1 1 586BBAA5
+P 10650 4700
+F 0 "#FLG05" H 10650 4795 50  0001 C CNN
+F 1 "PWR_FLAG" H 10650 4880 50  0000 C CNN
+F 2 "" H 10650 4700 60  0000 C CNN
+F 3 "" H 10650 4700 60  0000 C CNN
+	1    10650 4700
+	1    0    0    1
+$EndComp
+$Comp
+L +12V #PWR06
+U 1 1 586BFF75
+P 10650 4700
+F 0 "#PWR06" H 10650 4550 50  0001 C CNN
+F 1 "+12V" H 10650 4840 50  0000 C CNN
+F 2 "" H 10650 4700 60  0000 C CNN
+F 3 "" H 10650 4700 60  0000 C CNN
+	1    10650 4700
+	1    0    0    -1
+$EndComp
+Wire Wire Line
+	10650 1350 10750 1350
+Connection ~ 10650 1250
+Text GLabel 10750 1450 0    60   Output ~ 0
++250VAC
 $EndSCHEMATC

Commit message: Digitized the real DSKY Indicator Driver Module schematic from ND-1021042
Parts:
- added C1, C2: 4.7uF, symbol CP1
- added C3, C4, C5, C6, C7: 0.1uF, symbol CP1
- added CR1, CR10, CR11, CR12, CR13, CR14, CR15, CR16, CR17, CR18, CR19, CR2, CR20, CR21, CR22, CR23, CR24, CR25, CR26, CR27, CR28, CR29, CR3, CR30, CR31, CR32, CR33, CR34, CR35, CR36, CR37, CR38, CR39, CR4, CR40, CR41, CR42, CR43, CR44, CR45, CR46, CR47, CR48, CR49, CR5, CR50, CR51, CR52, CR53, CR54, CR55, CR56, CR57, CR58, CR59, CR6, CR60, CR61, CR62, CR63, CR64, CR7, CR8, CR9: D, symbol D
- added K1, K10, K11, K12, K13, K14, K15, K16, K17, K18, K19, K2, K20, K3, K4, K5, K6, K7, K8, K9: EC2-12TNU, symbol EC2-12TNU
- added K21, K22: EC2-12NU, symbol EC2-12NU
- added L1, L2: 8.2uH, symbol INDUCTOR
- added Q1, Q10, Q11, Q12, Q13, Q8, Q9: PN2907A, symbol Q_PNP_EBC
- added Q2, Q3, Q4, Q5, Q6, Q7: PN2222A, symbol Q_NPN_EBC
- added R1, R11, R12, R15, R16, R19, R2, R22, R24, R3, R4, R6, R7, R9: 10k, symbol R
- added R10, R5, R8: 18k, symbol R
- added R101, R102, R103, R104, R105, R106, R107, R108, R109, R110, R111, R112, R113, R114, R115, R116, R117, R118, R119, R120, R121, R122, R123, R124, R125, R126, R127, R128, R129, R130, R131, R132, R133, R134, R135, R136, R137, R138, R139, R140, R141, R142: 1.5k, symbol R
- added R13, R17: 20k, symbol R
- added R14, R18, R21, R23: 2k, symbol R
- added R20, R25: 1k, symbol R
Connections:
- net labels added: +28VDC, P1, P10, P100, P101, P102, P103, P104, P106, P107, P108, P109, P11, P110, P111, P113, P114, P115, P116, P117, P118, P119, P12, P120, P121, P122, P123, P124, P13, P14, P15, P16, P17, P18, P19, P2, P20, P21, P22, P23, P24, P25, P26, P27, P28, P29, P3, P30, P31, P32, P33, P34, P35, P36, P37, P38, P39, P4, P40, P41, P42, P43, P44, P45, P46, P47, P48, P49, P5, P50, P51, P52, P53, P54, P55, P56, P57, P58, P59, P6, P60, P61, P62, P63, P64, P65, P66, P67, P69, P7, P70, P71, P72, P73, P74, P75, P76, P77, P78, P79, P8, P80, P81, P82, P83, P84, P85, P86, P87, P88, P89, P9, P90, P91, P92, P94, P95, P97, P98, P99
- net labels removed: +12V, +250VAC, DEC12_LINE/, DEC1_R1_R, DEC1_R1_S, DEC1_R2_R, DEC1_R2_S, DEC1_R3_R, DEC1_R3_S, DEC1_R4_R, DEC1_R4_S, DEC1_R5_R, DEC1_R5_S, DEC1_SEGA, DEC1_SEGB, DEC1_SEGC, DEC1_SEGD, DEC1_SEGE, DEC1_SEGF, DEC1_SEGG, DEC2_R1_R, DEC2_R1_S, DEC2_R2_R, DEC2_R2_S, DEC2_R3_R, DEC2_R3_S, DEC2_R4_R, DEC2_R4_S, DEC2_R5_R, DEC2_R5_S, DEC2_SEGA, DEC2_SEGB, DEC2_SEGC, DEC2_SEGD, DEC2_SEGE, DEC2_SEGF, DEC2_SEGG, DEC3_LINE/, DEC3_R1_R, DEC3_R1_S, DEC3_R2_R, DEC3_R2_S, DEC3_R3_R, DEC3_R3_S, DEC3_R4_R, DEC3_R4_S, DEC3_R5_R, DEC3_R5_S, DEC3_SEGA, DEC3_SEGB, DEC3_SEGC, DEC3_SEGD, DEC3_SEGE, DEC3_SEGF, DEC3_SEGG, DEC4_LINE145/, DEC4_LINE2/, DEC4_LINE3/, DEC4_R15_IN, DEC4_R1_R, DEC4_R1_S, DEC4_R2_OUT, DEC4_R2_R, DEC4_R2_S, DEC4_R3_R, DEC4_R3_S, DEC4_R4_R, DEC4_R4_S, DEC4_R5_R, DEC4_R5_S, DEC4_SEGA, DEC4_SEGB, DEC4_SEGC, DEC4_SEGD, DEC4_SEGE, DEC4_SEGF, DEC4_SEGG, LINE1_ADDR1, LINE1_ADDR2, LINE1_ADDR3, LINE1_ADDR4, LINE2_ADDR1, LINE2_ADDR2, LINE2_ADDR3, LINE2_ADDR4, R21_C1, R21_C2, R21_NC1, R21_NC2, R21_NO1, R21_NO2, R21_S, R22_C1, R22_C2, R22_NC1, R22_NC2, R22_NO1, R22_NO2, R22_S, RELAY_BIT_1, RELAY_BIT_1/, RELAY_BIT_2, RELAY_BIT_2/, RELAY_BIT_3, RELAY_BIT_3/, RELAY_LINE_1, RELAY_LINE_2, RELAY_SET_1, RELAY_SET_2, RELAY_SET_3
- wire segments 157 -> 666
- no-connect marks 0 -> 27
Other:
- note added: "0VDC"
- note added: "CKT\n000"
- note added: "CKT\n001"
- note added: "CKT\n002"
- note added: "CKT\n003"
- note added: "CKT\n004"
- note added: "CKT\n005"
- note added: "CKT\n006"
- note added: "CKT\n007"
- note added: "CKT\n008"
- note added: "CKT\n009"
- note added: "CKT\n011"
- note added: "EV250"
- note added: "OSGRD"
- note added: "X"
- note added: "Y"
- note removed: "Line Drivers"
- note removed: "Relay Drivers"
- note removed: "Relay Matrix"

Commit message: Redid the Keyboard Module according to ND-1021042 schematics. Also renumbered the DIN 41612 128P connector to make more DSKY sense
Parts:
- removed P1: DIN_41612_128P, symbol DIN_41612_128P
- added P1: PCN10A-128P, symbol PCN10A-128P
Connections:
- wire segments 666 -> 857

Commit message: Added PCN10A-128P and EC2-12NU footprints
Parts:
- C1, C2, C3, C4, C5, C6, C7: footprint (none) -> Capacitors_SMD:C_0603_HandSoldering
- CR1, CR10, CR11, CR12, CR13, CR14, CR15, CR16, CR17, CR18, CR19, CR2, CR20, CR21, CR22, CR23, CR24, CR25, CR26, CR27, CR28, CR29, CR3, CR30, CR31, CR32, CR33, CR34, CR35, CR36, CR37, CR38, CR39, CR4, CR40, CR41, CR42, CR43, CR44, CR45, CR46, CR47, CR48, CR49, CR5, CR50, CR51, CR52, CR53, CR54, CR55, CR56, CR57, CR58, CR59, CR6, CR60, CR61, CR62, CR63, CR64, CR7, CR8, CR9: footprint (none) -> Diodes_SMD:D_0603
- K1, K10, K11, K12, K13, K14, K15, K16, K17, K18, K19, K2, K20, K3, K4, K5, K6, K7, K8, K9: footprint (none) -> agc_footprints:EC2-12TNU
- K21, K22: footprint (none) -> agc_footprints:EC2-12NU
- L1, L2: footprint (none) -> Inductors:Inductor_1212
- P1: footprint (none) -> agc_footprints:PCN10A-128P
- Q1, Q10, Q11, Q12, Q13, Q2, Q3, Q4, Q5, Q6, Q7, Q8, Q9: footprint (none) -> TO_SOT_Packages_THT:TO-3
- R1, R10, R101, R102, R103, R104, R105, R106, R107, R108, R109, R11, R110, R111, R112, R113, R114, R115, R116, R117, R118, R119, R12, R120, R121, R122, R123, R124, R125, R126, R127, R128, R129, R13, R130, R131, R132, R133, R134, R135, R136, R137, R138, R139, R14, R140, R141, R142, R15, R16, R17, R18, R19, R2, R20, R21, R22, R23, R24, R25, R3, R4, R5, R6, R7, R8, R9: footprint (none) -> Resistors_SMD:R_0603_HandSoldering
Connections:
- wire segments 857 -> 666
