File: dsky/digital_indicator/digital_indicator.kicad_pcb (KiCad board)
At the start: 4 copper layers, 63.5 x 109.2 mm, 362 parts, among them P1 CONN_02X20, P2 CONN_02X20, P3 CONN_02X20, P4 CONN_02X20

Commit message: Rev. 1 of the Digital Indicator board
Parts:
- removed R100, R101, R102, R103, R104, R105, R106, R107, R108, R109, R110, R111, R112, R113, R114, R115, R116, R117, R118, R119, R120, R121, R122, R123, R124, R125, R126, R127, R128, R129, R130, R131, R132, R133, R134, R135, R136, R137, R138, R139, R14, R140, R141, R142, R143, R144, R145, R146, R147, R148, R149, R15, R150, R151, R152, R153, R154, R155, R156, R157, R158, R159, R16, R160, R161, R162, R163, R164, R165, R166, R167, R168, R169, R17, R170, R171, R172, R173, R174, R175, R176, R177, R178, R18, R19, R20, R21, R22, R23, R24, R25, R26, R27, R28, R29, R30, R31, R32, R33, R34, R35, R36, R37, R38, R39, R40, R41, R42, R43, R44, R45, R46, R47, R48, R49, R50, R51, R52, R53, R54, R55, R56, R57, R58, R59, R60, R61, R62, R63, R64, R65, R66, R67, R68, R69, R70, R71, R72, R73, R74, R75, R76, R77, R78, R79, R80, R81, R82, R83, R84, R85, R86, R87, R88, R89, R90, R91, R92, R93, R94, R95, R96, R97, R98, R99: 1k, Resistors_SMD:R_0603
- added RN10: R8_BUSSED, agc_footprints:R8_746, B.Cu at (153.9, 103.5)
- added RN11: R8_BUSSED, agc_footprints:R8_746, B.Cu at (164.0, 103.5)
- added RN12: R8_BUSSED, agc_footprints:R8_746, B.Cu at (123.4, 122.9)
- added RN13: R8_BUSSED, agc_footprints:R8_746, B.Cu at (133.6, 122.9)
- added RN14: R8_BUSSED, agc_footprints:R8_746, B.Cu at (143.8, 122.9)
- added RN15: R8_BUSSED, agc_footprints:R8_746, B.Cu at (153.9, 122.9)
- added RN16: R8_BUSSED, agc_footprints:R8_746, B.Cu at (164.0, 122.9)
- added RN17: R8_BUSSED, agc_footprints:R8_746, B.Cu at (123.4, 142.4)
- added RN18: R8_BUSSED, agc_footprints:R8_746, B.Cu at (133.6, 142.4)
- added RN19: R8_BUSSED, agc_footprints:R8_746, B.Cu at (143.8, 142.4)
- added RN2: R8_BUSSED, agc_footprints:R8_746, B.Cu at (164.0, 60.3)
- added RN20: R8_BUSSED, agc_footprints:R8_746, B.Cu at (153.9, 142.4)
- added RN21: R8_BUSSED, agc_footprints:R8_746, B.Cu at (164.0, 142.4)
- added RN3: R8_BUSSED, agc_footprints:R8_746, B.Cu at (117.9, 84.5)
- added RN4: R8_BUSSED, agc_footprints:R8_746, B.Cu at (128.0, 84.5)
- added RN5: R8_BUSSED, agc_footprints:R8_746, B.Cu at (153.9, 84.5)
- added RN6: R8_BUSSED, agc_footprints:R8_746, B.Cu at (164.0, 84.5)
- added RN7: R8_BUSSED, agc_footprints:R8_746, B.Cu at (123.4, 103.5)
- added RN8: R8_BUSSED, agc_footprints:R8_746, B.Cu at (133.6, 103.5)
- added RN9: R8_BUSSED, agc_footprints:R8_746, B.Cu at (143.8, 103.5)
- R1, R11, R5, R8: value 1k -> 250; moved to B.Cu
- R10, R13, R2, R3, R4, R7: value 1k -> 500; moved to B.Cu
- R12, R6, R9: moved to B.Cu
- moved R11 111.5 mm to (124.5, 127.0)
- moved R12 110.3 mm to (116.3, 137.9)
- moved R1 107.1 mm to (124.2, 52.3), turned to 180 degrees
- moved R13 106.0 mm to (116.3, 135.4)
- moved R9 105.7 mm to (116.3, 118.6)
- moved R7 104.0 mm to (116.3, 96.5)
- moved R6 102.0 mm to (116.3, 99.1), turned to 180 degrees
- moved R3 100.3 mm to (124.0, 69.1)
- moved R5 91.8 mm to (124.5, 88.9)
- moved R8 88.7 mm to (124.5, 108.0)
- moved R10 78.9 mm to (116.3, 115.8), turned to 180 degrees
- moved RN1 77.8 mm to (153.9, 60.3), turned to 270 degrees
- moved R4 42.2 mm to (160.8, 69.1)
- moved R2 30.2 mm to (160.3, 45.0), turned to 180 degrees
- moved P2 9.02 mm to (142.9, 90.2)
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Connections:
- D10 pad 1: Net-(D10-Pad1) -> MD1_D
- D10 pad 2: +12V -> Net-(D10-Pad2)
- D102 pad 1: Net-(D102-Pad1) -> R2D1_A
- D102 pad 2: +12V -> Net-(D102-Pad2)
- D103 pad 1: Net-(D103-Pad1) -> R2D1_B
- D103 pad 2: +12V -> Net-(D103-Pad2)
- D104 pad 1: Net-(D104-Pad1) -> R2D1_C
- D104 pad 2: +12V -> Net-(D104-Pad2)
- D105 pad 1: Net-(D105-Pad1) -> R2D1_D
- D105 pad 2: +12V -> Net-(D105-Pad2)
- D106 pad 1: Net-(D106-Pad1) -> R2D1_E
- D106 pad 2: +12V -> Net-(D106-Pad2)
- D107 pad 1: Net-(D107-Pad1) -> R2D1_F
- D107 pad 2: +12V -> Net-(D107-Pad2)
- D108 pad 1: Net-(D108-Pad1) -> R2D1_G
- D108 pad 2: +12V -> Net-(D108-Pad2)
- D109 pad 1: Net-(D109-Pad1) -> R2D2_A
- D109 pad 2: +12V -> Net-(D109-Pad2)
- D11 pad 1: Net-(D11-Pad1) -> MD1_E
- D11 pad 2: +12V -> Net-(D11-Pad2)
- D110 pad 1: Net-(D110-Pad1) -> R2D2_B
- D110 pad 2: +12V -> Net-(D110-Pad2)
- D111 pad 1: Net-(D111-Pad1) -> R2D2_C
- D111 pad 2: +12V -> Net-(D111-Pad2)
- D112 pad 1: Net-(D112-Pad1) -> R2D2_D
- D112 pad 2: +12V -> Net-(D112-Pad2)
- D113 pad 1: Net-(D113-Pad1) -> R2D2_E
- D113 pad 2: +12V -> Net-(D113-Pad2)
- D114 pad 1: Net-(D114-Pad1) -> R2D2_F
- D114 pad 2: +12V -> Net-(D114-Pad2)
- D115 pad 1: Net-(D115-Pad1) -> R2D2_G
- D115 pad 2: +12V -> Net-(D115-Pad2)
- D116 pad 1: Net-(D116-Pad1) -> R2D3_A
- D116 pad 2: +12V -> Net-(D116-Pad2)
- D117 pad 1: Net-(D117-Pad1) -> R2D3_B
- D117 pad 2: +12V -> Net-(D117-Pad2)
- D118 pad 1: Net-(D118-Pad1) -> R2D3_C
- D118 pad 2: +12V -> Net-(D118-Pad2)
- D119 pad 1: Net-(D119-Pad1) -> R2D3_D
- D119 pad 2: +12V -> Net-(D119-Pad2)
- D12 pad 1: Net-(D12-Pad1) -> MD1_F
- D12 pad 2: +12V -> Net-(D12-Pad2)
- D120 pad 1: Net-(D120-Pad1) -> R2D3_E
- D120 pad 2: +12V -> Net-(D120-Pad2)
- D121 pad 1: Net-(D121-Pad1) -> R2D3_F
- D121 pad 2: +12V -> Net-(D121-Pad2)
- D122 pad 1: Net-(D122-Pad1) -> R2D3_G
- D122 pad 2: +12V -> Net-(D122-Pad2)
- D123 pad 1: Net-(D123-Pad1) -> R2D4_A
- D123 pad 2: +12V -> Net-(D123-Pad2)
- D124 pad 1: Net-(D124-Pad1) -> R2D4_B
- D124 pad 2: +12V -> Net-(D124-Pad2)
- D125 pad 1: Net-(D125-Pad1) -> R2D4_C
- D125 pad 2: +12V -> Net-(D125-Pad2)
- D126 pad 1: Net-(D126-Pad1) -> R2D4_D
- D126 pad 2: +12V -> Net-(D126-Pad2)
- D127 pad 1: Net-(D127-Pad1) -> R2D4_E
- D127 pad 2: +12V -> Net-(D127-Pad2)
- D128 pad 1: Net-(D128-Pad1) -> R2D4_F
- D128 pad 2: +12V -> Net-(D128-Pad2)
- D129 pad 1: Net-(D129-Pad1) -> R2D4_G
- D129 pad 2: +12V -> Net-(D129-Pad2)
- D13 pad 1: Net-(D13-Pad1) -> MD1_G
- D13 pad 2: +12V -> Net-(D13-Pad2)
- D130 pad 1: Net-(D130-Pad1) -> R2D5_A
- D130 pad 2: +12V -> Net-(D130-Pad2)
- D131 pad 1: Net-(D131-Pad1) -> R2D5_B
- D131 pad 2: +12V -> Net-(D131-Pad2)
- D132 pad 1: Net-(D132-Pad1) -> R2D5_C
- D132 pad 2: +12V -> Net-(D132-Pad2)
- D133 pad 1: Net-(D133-Pad1) -> R2D5_D
- D133 pad 2: +12V -> Net-(D133-Pad2)
- D134 pad 1: Net-(D134-Pad1) -> R2D5_E
- D134 pad 2: +12V -> Net-(D134-Pad2)
- D135 pad 1: Net-(D135-Pad1) -> R2D5_F
- D135 pad 2: +12V -> Net-(D135-Pad2)
- D136 pad 1: Net-(D136-Pad1) -> R2D5_G
- D136 pad 2: +12V -> Net-(D136-Pad2)
- D138 pad 1: Net-(D138-Pad1) -> Net-(D137-Pad1)
- D139 pad 1: Net-(D139-Pad1) -> Net-(D137-Pad1)
- D14 pad 1: Net-(D14-Pad1) -> MD2_A
- D14 pad 2: +12V -> Net-(D14-Pad2)
- D140 pad 1: Net-(D140-Pad1) -> Net-(D137-Pad1)
- D143 pad 1: Net-(D143-Pad1) -> Net-(D141-Pad1)
- D144 pad 1: Net-(D144-Pad1) -> R3D1_A
- D144 pad 2: +12V -> Net-(D144-Pad2)
- D145 pad 1: Net-(D145-Pad1) -> R3D1_B
- D145 pad 2: +12V -> Net-(D145-Pad2)
- D146 pad 1: Net-(D146-Pad1) -> R3D1_C
- D146 pad 2: +12V -> Net-(D146-Pad2)
- D147 pad 1: Net-(D147-Pad1) -> R3D1_D
- D147 pad 2: +12V -> Net-(D147-Pad2)
- D148 pad 1: Net-(D148-Pad1) -> R3D1_E
- D148 pad 2: +12V -> Net-(D148-Pad2)
- D149 pad 1: Net-(D149-Pad1) -> R3D1_F
- D149 pad 2: +12V -> Net-(D149-Pad2)
- D15 pad 1: Net-(D15-Pad1) -> MD2_B
- D15 pad 2: +12V -> Net-(D15-Pad2)
- D150 pad 1: Net-(D150-Pad1) -> R3D1_G
- D150 pad 2: +12V -> Net-(D150-Pad2)
- D151 pad 1: Net-(D151-Pad1) -> R3D2_A
- D151 pad 2: +12V -> Net-(D151-Pad2)
- D152 pad 1: Net-(D152-Pad1) -> R3D2_B
- D152 pad 2: +12V -> Net-(D152-Pad2)
- D153 pad 1: Net-(D153-Pad1) -> R3D2_C
- D153 pad 2: +12V -> Net-(D153-Pad2)
- D154 pad 1: Net-(D154-Pad1) -> R3D2_D
- D154 pad 2: +12V -> Net-(D154-Pad2)
- D155 pad 1: Net-(D155-Pad1) -> R3D2_E
- D155 pad 2: +12V -> Net-(D155-Pad2)
- D156 pad 1: Net-(D156-Pad1) -> R3D2_F
- D156 pad 2: +12V -> Net-(D156-Pad2)
- D157 pad 1: Net-(D157-Pad1) -> R3D2_G
- D157 pad 2: +12V -> Net-(D157-Pad2)
- D158 pad 1: Net-(D158-Pad1) -> R3D3_A
- D158 pad 2: +12V -> Net-(D158-Pad2)
- D159 pad 1: Net-(D159-Pad1) -> R3D3_B
- D159 pad 2: +12V -> Net-(D159-Pad2)
- D16 pad 1: Net-(D16-Pad1) -> MD2_C
- D16 pad 2: +12V -> Net-(D16-Pad2)
- D160 pad 1: Net-(D160-Pad1) -> R3D3_C
- D160 pad 2: +12V -> Net-(D160-Pad2)
- D161 pad 1: Net-(D161-Pad1) -> R3D3_D
- D161 pad 2: +12V -> Net-(D161-Pad2)
- D162 pad 1: Net-(D162-Pad1) -> R3D3_E
- D162 pad 2: +12V -> Net-(D162-Pad2)
- D163 pad 1: Net-(D163-Pad1) -> R3D3_F
- D163 pad 2: +12V -> Net-(D163-Pad2)
- D164 pad 1: Net-(D164-Pad1) -> R3D3_G
- D164 pad 2: +12V -> Net-(D164-Pad2)
- D165 pad 1: Net-(D165-Pad1) -> R3D4_A
- D165 pad 2: +12V -> Net-(D165-Pad2)
- D166 pad 1: Net-(D166-Pad1) -> R3D4_B
- D166 pad 2: +12V -> Net-(D166-Pad2)
- D167 pad 1: Net-(D167-Pad1) -> R3D4_C
- D167 pad 2: +12V -> Net-(D167-Pad2)
- D168 pad 1: Net-(D168-Pad1) -> R3D4_D
- D168 pad 2: +12V -> Net-(D168-Pad2)
- D169 pad 1: Net-(D169-Pad1) -> R3D4_E
- D169 pad 2: +12V -> Net-(D169-Pad2)
- D17 pad 1: Net-(D17-Pad1) -> MD2_D
- D17 pad 2: +12V -> Net-(D17-Pad2)
- D170 pad 1: Net-(D170-Pad1) -> R3D4_F
- D170 pad 2: +12V -> Net-(D170-Pad2)
- D171 pad 1: Net-(D171-Pad1) -> R3D4_G
- D171 pad 2: +12V -> Net-(D171-Pad2)
- D172 pad 1: Net-(D172-Pad1) -> R3D5_A
- D172 pad 2: +12V -> Net-(D172-Pad2)
- D173 pad 1: Net-(D173-Pad1) -> R3D5_B
- D173 pad 2: +12V -> Net-(D173-Pad2)
- D174 pad 1: Net-(D174-Pad1) -> R3D5_C
- D174 pad 2: +12V -> Net-(D174-Pad2)
- D175 pad 1: Net-(D175-Pad1) -> R3D5_D
- D175 pad 2: +12V -> Net-(D175-Pad2)
- D176 pad 1: Net-(D176-Pad1) -> R3D5_E
- D176 pad 2: +12V -> Net-(D176-Pad2)
- D177 pad 1: Net-(D177-Pad1) -> R3D5_F
- D177 pad 2: +12V -> Net-(D177-Pad2)
- D178 pad 1: Net-(D178-Pad1) -> R3D5_G
- D178 pad 2: +12V -> Net-(D178-Pad2)
- D18 pad 1: Net-(D18-Pad1) -> MD2_E
- D18 pad 2: +12V -> Net-(D18-Pad2)
- D19 pad 1: Net-(D19-Pad1) -> MD2_F
- D19 pad 2: +12V -> Net-(D19-Pad2)
- D2 pad 1: Net-(D2-Pad1) -> Net-(D1-Pad1)
- D20 pad 1: Net-(D20-Pad1) -> MD2_G
- D20 pad 2: +12V -> Net-(D20-Pad2)
- D22 pad 1: Net-(D22-Pad1) -> Net-(D21-Pad1)
- D23 pad 1: Net-(D23-Pad1) -> VD1_A
- D23 pad 2: +12V -> Net-(D23-Pad2)
- D24 pad 1: Net-(D24-Pad1) -> VD1_B
- D24 pad 2: +12V -> Net-(D24-Pad2)
- D25 pad 1: Net-(D25-Pad1) -> VD1_C
- D25 pad 2: +12V -> Net-(D25-Pad2)
- D26 pad 1: Net-(D26-Pad1) -> VD1_D
- D26 pad 2: +12V -> Net-(D26-Pad2)
- D27 pad 1: Net-(D27-Pad1) -> VD1_E
- D27 pad 2: +12V -> Net-(D27-Pad2)
- D28 pad 1: Net-(D28-Pad1) -> VD1_F
- D28 pad 2: +12V -> Net-(D28-Pad2)
- D29 pad 1: Net-(D29-Pad1) -> VD1_G
- D29 pad 2: +12V -> Net-(D29-Pad2)
- D3 pad 1: Net-(D3-Pad1) -> Net-(D1-Pad1)
- D30 pad 1: Net-(D30-Pad1) -> VD2_A
- D30 pad 2: +12V -> Net-(D30-Pad2)
- D31 pad 1: Net-(D31-Pad1) -> VD2_B
- D31 pad 2: +12V -> Net-(D31-Pad2)
- D32 pad 1: Net-(D32-Pad1) -> VD2_C
- D32 pad 2: +12V -> Net-(D32-Pad2)
- D33 pad 1: Net-(D33-Pad1) -> VD2_D
- D33 pad 2: +12V -> Net-(D33-Pad2)
- D34 pad 1: Net-(D34-Pad1) -> VD2_E
- D34 pad 2: +12V -> Net-(D34-Pad2)
- D35 pad 1: Net-(D35-Pad1) -> VD2_F
- D35 pad 2: +12V -> Net-(D35-Pad2)
- D36 pad 1: Net-(D36-Pad1) -> VD2_G
- D36 pad 2: +12V -> Net-(D36-Pad2)
- D38 pad 1: Net-(D38-Pad1) -> Net-(D37-Pad1)
- D39 pad 1: Net-(D39-Pad1) -> ND1_A
- D39 pad 2: +12V -> Net-(D39-Pad2)
- D4 pad 1: Net-(D4-Pad1) -> Net-(D1-Pad1)
- D40 pad 1: Net-(D40-Pad1) -> ND1_B
- D40 pad 2: +12V -> Net-(D40-Pad2)
- D41 pad 1: Net-(D41-Pad1) -> ND1_C
- D41 pad 2: +12V -> Net-(D41-Pad2)
- D42 pad 1: Net-(D42-Pad1) -> ND1_D
- D42 pad 2: +12V -> Net-(D42-Pad2)
- D43 pad 1: Net-(D43-Pad1) -> ND1_E
- D43 pad 2: +12V -> Net-(D43-Pad2)
- D44 pad 1: Net-(D44-Pad1) -> ND1_F
- D44 pad 2: +12V -> Net-(D44-Pad2)
- D45 pad 1: Net-(D45-Pad1) -> ND1_G
- D45 pad 2: +12V -> Net-(D45-Pad2)
- D46 pad 1: Net-(D46-Pad1) -> ND2_A
- D46 pad 2: +12V -> Net-(D46-Pad2)
- D47 pad 1: Net-(D47-Pad1) -> ND2_B
- D47 pad 2: +12V -> Net-(D47-Pad2)
- D48 pad 1: Net-(D48-Pad1) -> ND2_C
- D48 pad 2: +12V -> Net-(D48-Pad2)
- D49 pad 1: Net-(D49-Pad1) -> ND2_D
- D49 pad 2: +12V -> Net-(D49-Pad2)
- D50 pad 1: Net-(D50-Pad1) -> ND2_E
- D50 pad 2: +12V -> Net-(D50-Pad2)
- D51 pad 1: Net-(D51-Pad1) -> ND2_F
- D51 pad 2: +12V -> Net-(D51-Pad2)
- D52 pad 1: Net-(D52-Pad1) -> ND2_G
- D52 pad 2: +12V -> Net-(D52-Pad2)
- D54 pad 1: Net-(D54-Pad1) -> Net-(D53-Pad1)
- D55 pad 1: Net-(D55-Pad1) -> Net-(D53-Pad1)
- D56 pad 1: Net-(D56-Pad1) -> Net-(D53-Pad1)
- D59 pad 1: Net-(D59-Pad1) -> Net-(D57-Pad1)
- D6 pad 1: Net-(D6-Pad1) -> Net-(D5-Pad1)
- D60 pad 1: Net-(D60-Pad1) -> R1D1_A
- D60 pad 2: +12V -> Net-(D60-Pad2)
- D61 pad 1: Net-(D61-Pad1) -> R1D1_B
- D61 pad 2: +12V -> Net-(D61-Pad2)
- D62 pad 1: Net-(D62-Pad1) -> R1D1_C
- D62 pad 2: +12V -> Net-(D62-Pad2)
- D63 pad 1: Net-(D63-Pad1) -> R1D1_D
- D63 pad 2: +12V -> Net-(D63-Pad2)
- D64 pad 1: Net-(D64-Pad1) -> R1D1_E
- D64 pad 2: +12V -> Net-(D64-Pad2)
- D65 pad 1: Net-(D65-Pad1) -> R1D1_F
- D65 pad 2: +12V -> Net-(D65-Pad2)
- D66 pad 1: Net-(D66-Pad1) -> R1D1_G
- D66 pad 2: +12V -> Net-(D66-Pad2)
- D67 pad 1: Net-(D67-Pad1) -> R1D2_A
- D67 pad 2: +12V -> Net-(D67-Pad2)
- D68 pad 1: Net-(D68-Pad1) -> R1D2_B
- D68 pad 2: +12V -> Net-(D68-Pad2)
- D69 pad 1: Net-(D69-Pad1) -> R1D2_C
- D69 pad 2: +12V -> Net-(D69-Pad2)
- D7 pad 1: Net-(D7-Pad1) -> MD1_A
- D7 pad 2: +12V -> Net-(D7-Pad2)
- D70 pad 1: Net-(D70-Pad1) -> R1D2_D
- D70 pad 2: +12V -> Net-(D70-Pad2)
- D71 pad 1: Net-(D71-Pad1) -> R1D2_E
- D71 pad 2: +12V -> Net-(D71-Pad2)
- D72 pad 1: Net-(D72-Pad1) -> R1D2_F
- D72 pad 2: +12V -> Net-(D72-Pad2)
- D73 pad 1: Net-(D73-Pad1) -> R1D2_G
- D73 pad 2: +12V -> Net-(D73-Pad2)
- D74 pad 1: Net-(D74-Pad1) -> R1D3_A
- D74 pad 2: +12V -> Net-(D74-Pad2)
- D75 pad 1: Net-(D75-Pad1) -> R1D3_B
- D75 pad 2: +12V -> Net-(D75-Pad2)
- D76 pad 1: Net-(D76-Pad1) -> R1D3_C
- D76 pad 2: +12V -> Net-(D76-Pad2)
- D77 pad 1: Net-(D77-Pad1) -> R1D3_D
- D77 pad 2: +12V -> Net-(D77-Pad2)
- D78 pad 1: Net-(D78-Pad1) -> R1D3_E
- D78 pad 2: +12V -> Net-(D78-Pad2)
- D79 pad 1: Net-(D79-Pad1) -> R1D3_F
- D79 pad 2: +12V -> Net-(D79-Pad2)
- D8 pad 1: Net-(D8-Pad1) -> MD1_B
- D8 pad 2: +12V -> Net-(D8-Pad2)
- D80 pad 1: Net-(D80-Pad1) -> R1D3_G
- D80 pad 2: +12V -> Net-(D80-Pad2)
- D81 pad 1: Net-(D81-Pad1) -> R1D4_A
- D81 pad 2: +12V -> Net-(D81-Pad2)
- D82 pad 1: Net-(D82-Pad1) -> R1D4_B
- D82 pad 2: +12V -> Net-(D82-Pad2)
- D83 pad 1: Net-(D83-Pad1) -> R1D4_C
- D83 pad 2: +12V -> Net-(D83-Pad2)
- D84 pad 1: Net-(D84-Pad1) -> R1D4_D
- D84 pad 2: +12V -> Net-(D84-Pad2)
- D85 pad 1: Net-(D85-Pad1) -> R1D4_E
- D85 pad 2: +12V -> Net-(D85-Pad2)
- D86 pad 1: Net-(D86-Pad1) -> R1D4_F
- D86 pad 2: +12V -> Net-(D86-Pad2)
- D87 pad 1: Net-(D87-Pad1) -> R1D4_G
- D87 pad 2: +12V -> Net-(D87-Pad2)
- D88 pad 1: Net-(D88-Pad1) -> R1D5_A
- D88 pad 2: +12V -> Net-(D88-Pad2)
- D89 pad 1: Net-(D89-Pad1) -> R1D5_B
- D89 pad 2: +12V -> Net-(D89-Pad2)
- D9 pad 1: Net-(D9-Pad1) -> MD1_C
- D9 pad 2: +12V -> Net-(D9-Pad2)
- D90 pad 1: Net-(D90-Pad1) -> R1D5_C
- D90 pad 2: +12V -> Net-(D90-Pad2)
- D91 pad 1: Net-(D91-Pad1) -> R1D5_D
- D91 pad 2: +12V -> Net-(D91-Pad2)
- D92 pad 1: Net-(D92-Pad1) -> R1D5_E
- D92 pad 2: +12V -> Net-(D92-Pad2)
- D93 pad 1: Net-(D93-Pad1) -> R1D5_F
- D93 pad 2: +12V -> Net-(D93-Pad2)
- D94 pad 1: Net-(D94-Pad1) -> R1D5_G
- D94 pad 2: +12V -> Net-(D94-Pad2)
- D96 pad 1: Net-(D96-Pad1) -> Net-(D95-Pad1)
- D97 pad 1: Net-(D97-Pad1) -> Net-(D95-Pad1)
- D98 pad 1: Net-(D98-Pad1) -> Net-(D95-Pad1)
- D99 pad 1: Net-(D99-Pad1) -> Net-(D101-Pad1)
- P1 pad 1: COMACT -> ND2_A
- P1 pad 10: VD2_C -> MD2_E
- P1 pad 11: MD1_E -> ND2_F
- P1 pad 12: VD2_D -> MD2_F
- P1 pad 13: MD1_F -> ND2_G
- P1 pad 14: VD2_E -> MD2_G
- P1 pad 15: MD1_G -> ND1_A
- P1 pad 16: VD2_F -> MD1_A
- P1 pad 17: MD2_A -> ND1_B
- P1 pad 18: VD2_G -> MD1_B
- P1 pad 19: MD2_B -> ND1_C
- P1 pad 2: VD1_F -> MD2_A
- P1 pad 20: ND1_A -> MD1_C
- P1 pad 21: MD2_C -> ND1_D
- P1 pad 22: ND1_B -> MD1_D
- P1 pad 23: MD2_D -> ND1_E
- P1 pad 24: ND1_C -> MD1_E
- P1 pad 25: MD2_E -> ND1_F
- P1 pad 26: R1D3_F -> MD1_F
- P1 pad 27: MD2_F -> ND1_G
- P1 pad 28: R1D3_G -> MD1_G
- P1 pad 29: MD2_G -> VD1_C
- P1 pad 3: MD1_A -> ND2_B
- P1 pad 30: R1D4_A -> VD1_B
- P1 pad 31: VD1_A -> VD1_D
- P1 pad 32: R1D4_B -> VD1_A
- P1 pad 33: VD1_B -> VD1_E
- P1 pad 34: R1D4_C -> VD1_F
- P1 pad 35: VD1_C -> VD1_G
- P1 pad 36: R1D4_D -> +12V
- P1 pad 37: VD1_D -> VD2_B
- P1 pad 38: R1D4_E -> GND
- P1 pad 39: VD1_E -> VD2_A
- P1 pad 4: VD1_G -> MD2_B
- P1 pad 40: R1D4_F -> COMACT
- P1 pad 5: MD1_B -> ND2_C
- P1 pad 6: VD2_A -> MD2_C
- P1 pad 7: MD1_C -> ND2_D
- P1 pad 8: VD2_B -> MD2_D
- P1 pad 9: MD1_D -> ND2_E
- P2 pad 1: R2- -> R1D5_C
- P2 pad 10: R2D4_B -> R1D4_A
- P2 pad 11: R2D1_D -> R1D4_D
- P2 pad 12: R2D4_C -> R1D4_F
- P2 pad 13: R2D1_E -> R1D4_E
- P2 pad 14: R2D4_D -> +12V
- P2 pad 15: R2D1_F -> R1D4_G
- P2 pad 16: R2D4_E -> R1D3_B
- P2 pad 17: R2D1_G -> R1D3_C
- P2 pad 18: R2D4_F -> R1D3_A
- P2 pad 19: R2D2_A -> R1D3_D
- P2 pad 2: R2D3_E -> R1D5_B
- P2 pad 20: R2D4_G -> R1D3_F
- P2 pad 21: R2D2_B -> R1D3_E
- P2 pad 22: R2D5_A -> +12V
- P2 pad 23: R2D2_C -> R1D3_G
- P2 pad 24: R2D5_B -> R1D2_B
- P2 pad 25: R2D2_D -> R1D2_C
- P2 pad 26: R2D5_C -> R1D2_A
- P2 pad 27: R2D2_E -> R1D2_D
- P2 pad 28: R2D5_D -> R1D2_F
- P2 pad 29: R2D2_F -> R1D2_E
- P2 pad 3: R2+ -> R1D5_D
- P2 pad 30: R2D5_E -> R1D1_B
- P2 pad 31: R2D2_G -> R1D2_G
- P2 pad 32: R2D5_F -> R1D1_A
- P2 pad 33: R2D3_A -> R1D1_E
- P2 pad 34: R2D5_G -> R1D1_F
- P2 pad 35: R2D3_B -> R1D1_G
- P2 pad 36: Net-(P2-Pad36) -> VD2_E
- P2 pad 37: R2D3_C -> VD2_C
- P2 pad 38: Net-(P2-Pad38) -> VD2_F
- P2 pad 39: R2D3_D -> VD2_D
- P2 pad 4: R2D3_F -> R1D5_A
- P2 pad 40: Net-(P2-Pad40) -> VD2_G
- P2 pad 5: R2D1_A -> R1D5_E
- P2 pad 6: R2D3_G -> R1D5_F
- P2 pad 7: R2D1_B -> R1D5_G
- P2 pad 8: R2D4_A -> R1D4_B
- P2 pad 9: R2D1_C -> R1D4_C
- P3 pad 1: ND2_E -> R2D5_C
- P3 pad 10: ND1_D -> R2D4_B
- P3 pad 11: R1D1_A -> R2D4_D
- P3 pad 12: ND1_E -> R2D4_A
- P3 pad 13: R1D1_B -> R2D4_E
- P3 pad 14: ND1_F -> R2D4_F
- P3 pad 15: R1D1_C -> R2D3_C
- P3 pad 16: ND1_G -> R2D3_B
- P3 pad 17: R1D1_D -> R2D3_D
- P3 pad 18: ND2_A -> R2D3_A
- P3 pad 19: R1D1_E -> R2D3_E
- P3 pad 2: R1D3_B -> R2D5_B
- P3 pad 20: ND2_B -> R2D3_F
- P3 pad 21: R1D1_F -> R2D2_G
- P3 pad 22: ND2_C -> R2D3_G
- P3 pad 23: R1D1_G -> R2D2_C
- P3 pad 24: ND2_D -> R2D2_B
- P3 pad 25: R1D2_A -> R2D2_D
- P3 pad 26: R1D4_G -> R2D2_A
- P3 pad 27: R1D2_B -> R2D2_E
- P3 pad 28: R1D5_A -> R2D2_F
- P3 pad 29: R1D2_C -> R2D1_C
- P3 pad 3: ND2_F -> R2D5_D
- P3 pad 30: R1D5_B -> R2D1_B
- P3 pad 31: R1D2_D -> R2D1_D
- P3 pad 32: R1D5_C -> R2D1_A
- P3 pad 33: R1D2_E -> R2D1_E
- P3 pad 34: R1D5_D -> R2D1_F
- P3 pad 35: R1D2_F -> R2D1_G
- P3 pad 36: R1D5_E -> R1D1_C
- P3 pad 37: R1D2_G -> +12V
- P3 pad 38: R1D5_F -> R1D1_D
- P3 pad 39: R1D3_A -> R1-
- P3 pad 4: R1D3_C -> R2D5_A
- P3 pad 40: R1D5_G -> R1+
- P3 pad 5: ND2_G -> R2D5_E
- P3 pad 6: R1D3_D -> R2D5_F
- P3 pad 7: R1- -> R2D5_G
- P3 pad 8: R1D3_E -> R2D4_G
- P3 pad 9: R1+ -> R2D4_C
- P4 pad 1: R3- -> R3D5_C
- P4 pad 10: R3D2_A -> R3D4_B
- P4 pad 11: R3D2_C -> R3D4_D
- P4 pad 12: R3D2_B -> R3D4_A
- P4 pad 13: R3D2_D -> R3D4_E
- P4 pad 14: R3D2_F -> R3D4_F
- P4 pad 15: R3D2_E -> R3D3_C
- P4 pad 16: R3D2_G -> R3D3_B
- P4 pad 17: R3D3_C -> R3D3_D
- P4 pad 19: R3D3_D -> R3D3_E
- P4 pad 2: R3+ -> R3D5_B
- P4 pad 20: R3D3_B -> R3D3_F
- P4 pad 21: R3D3_E -> R3D3_G
- P4 pad 22: R3D3_F -> R3D2_G
- P4 pad 23: R3D3_G -> R3D2_C
- P4 pad 24: R3D4_A -> R3D2_B
- P4 pad 25: R3D4_C -> R3D2_D
- P4 pad 26: R3D4_B -> R3D2_A
- P4 pad 27: R3D4_D -> R3D2_E
- P4 pad 28: R3D4_F -> R3D2_F
- P4 pad 29: R3D4_E -> R3D1_C
- P4 pad 3: R3D1_C -> R3D5_D
- P4 pad 30: R3D4_G -> R3D1_B
- P4 pad 31: R3D5_C -> R3D1_D
- P4 pad 32: R3D5_A -> R3D1_A
- P4 pad 33: R3D5_D -> R3D1_E
- P4 pad 34: R3D5_B -> R3D1_F
- P4 pad 35: R3D5_E -> R3D1_G
- P4 pad 36: R3D5_F -> R3+
- P4 pad 37: R3D5_G -> R3-
- P4 pad 38: +12V -> R2+
- P4 pad 4: R3D1_A -> R3D5_A
- P4 pad 40: GND -> R2-
- P4 pad 5: R3D1_D -> R3D5_E
- P4 pad 6: R3D1_B -> R3D5_F
- P4 pad 7: R3D1_E -> R3D5_G
- P4 pad 8: R3D1_F -> R3D4_G
- P4 pad 9: R3D1_G -> R3D4_C
- R10 pad 1: MD1_D -> Net-(D101-Pad1)
- R10 pad 2: Net-(D10-Pad1) -> R2+
- R11 pad 1: MD1_E -> GND
- R11 pad 2: Net-(D11-Pad1) -> Net-(D137-Pad1)
- R12 pad 1: MD1_F -> Net-(D142-Pad1)
- R12 pad 2: Net-(D12-Pad1) -> R3-
- R13 pad 1: MD1_G -> Net-(D141-Pad1)
- R13 pad 2: Net-(D13-Pad1) -> R3+
- R2 pad 1: COMACT -> GND
- R2 pad 2: Net-(D2-Pad1) -> Net-(D5-Pad1)
- R3 pad 1: COMACT -> GND
- R3 pad 2: Net-(D3-Pad1) -> Net-(D21-Pad1)
- R4 pad 1: COMACT -> GND
- R4 pad 2: Net-(D4-Pad1) -> Net-(D37-Pad1)
- R5 pad 2: Net-(D5-Pad1) -> Net-(D53-Pad1)
- R6 pad 1: GND -> Net-(D58-Pad1)
- R6 pad 2: Net-(D6-Pad1) -> R1-
- R7 pad 1: MD1_A -> Net-(D57-Pad1)
- R7 pad 2: Net-(D7-Pad1) -> R1+
- R8 pad 1: MD1_B -> GND
- R8 pad 2: Net-(D8-Pad1) -> Net-(D95-Pad1)
- R9 pad 1: MD1_C -> Net-(D100-Pad1)
- R9 pad 2: Net-(D9-Pad1) -> R2-
- RN1 pad 1: Net-(RN1-Pad1) -> Net-(D13-Pad2)
- RN1 pad 10: Net-(RN1-Pad10) -> +12V
- RN1 pad 2: Net-(RN1-Pad2) -> Net-(D7-Pad2)
- RN1 pad 3: Net-(RN1-Pad3) -> Net-(D8-Pad2)
- RN1 pad 4: Net-(RN1-Pad4) -> Net-(D9-Pad2)
- RN1 pad 5: Net-(RN1-Pad5) -> +12V
- RN1 pad 6: Net-(RN1-Pad6) -> Net-(D10-Pad2)
- RN1 pad 7: Net-(RN1-Pad7) -> Net-(D11-Pad2)
- RN1 pad 8: Net-(RN1-Pad8) -> Net-(D12-Pad2)
- RN1 pad 9: Net-(RN1-Pad9) -> (no net)
Routing:
- net +12V: track 0.00 -> 110.9 mm, vias 0 -> 72
- net Net-(D137-Pad1): track 0.00 -> 51.4 mm, vias 0 -> 2
- net Net-(D53-Pad1): track 0.00 -> 43.9 mm, vias 0 -> 1
- net Net-(D95-Pad1): track 0.00 -> 35.7 mm, vias 0 -> 1
- net MD2_B: track 0.00 -> 29.6 mm, vias 0 -> 1
- net Net-(D1-Pad1): track 0.00 -> 25.7 mm, vias 0 -> 1
- net VD1_D: track 0.00 -> 25.1 mm, vias 0 -> 1
- net MD2_A: track 0.00 -> 25.0 mm, vias 0 -> 1
- net R2+: track 0.00 -> 24.8 mm
- net MD1_B: track 0.00 -> 24.3 mm, vias 0 -> 1
- net MD2_F: track 0.00 -> 24.2 mm, vias 0 -> 1
- net MD2_G: track 0.00 -> 23.9 mm, vias 0 -> 1
- net VD1_E: track 0.00 -> 23.7 mm, vias 0 -> 1
- net MD1_A: track 0.00 -> 23.5 mm, vias 0 -> 1
- net MD1_G: track 0.00 -> 22.5 mm, vias 0 -> 1
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- added copper zone on In2.Cu, net +12V
- added copper zone on In1.Cu, net GND
- removed copper zone on F.Cu, net +12V
Other:
- net class Default: clearance 0.2 -> 0.2032; trace_width 0.25 -> 0.2032; via_dia 0.8 -> 0.6096; via_drill 0.4 -> 0.3048
- net class Power added: clearance 0.2032, trace_width 0.508, via_dia 0.6096, via_drill 0.3048
- rule trace_clearance: 0.2 -> 0.2032
- rule trace_min: 0.2 -> 0.1524
- rule via_min_drill: 0.3 -> 0.3048
- rule via_min_size: 0.4 -> 0.6096
- board text added: "4/15/17"
- board text added: "DSKY Digital Indicator, Rev. 1"
