File: memory_timing_addressing/a14_1.sch (KiCad schematic (older format))
At the start: 22 parts, among them U14001 74HC02, U14002 74HC27, U14003 74HC04, U14004 74HC27, U14005 74HC02, U14006 74HC27, U14007 74HC02, U14008 74HC04, U14009 74HC27, U14010 74HC02, U14011 74HC02, U14012 74HC04, U14013 74HC27, U14014 74LVC07, U14015 74HC4002, U14016 74HC27, U14017 74HC02, U14018 74HC02, U14019 74HC27, U14020 74HC02

Commit message: Finished off and integrated module 14. Also fixed a couple of bugs this turned up (both initial conditions, and bad wiring in the CGMC pulse generator and S register)
Parts:
- removed unit 3 of U14012
- added R14003, R14004: 5k, symbol R
- added unit 6 of U14012
- added unit 5 of U14014
- added unit 6 of U14014
- added unit 4 of U14020
- added U14021, U14023, U14024, U14029, U14032: 74HC27, symbol 74HC27
- added U14022, U14025, U14027, U14030, U14031, U14060: 74HC02, symbol 74HC02
- added U14026: 74HC4002, symbol 74HC4002
- added U14028: 74HC04, symbol 74HC04
- added U14033: 74LVC07, symbol 74LVC07
- U14020: Initial (none) -> 1
Connections:
- net CLROPE: now also U14060.1
- net GND: now also U14012.7 (GND), U14014.7 (GND), U14014.7 (GND), U14020.7 (GND), U14021.7 (GND), U14021.7 (GND), U14021.7 (GND), U14022.7 (GND), U14022.7 (GND), U14022.7 (GND), U14022.7 (GND), U14023.7 (GND), U14023.7 (GND), U14023.7 (GND), U14024.7 (GND), U14024.7 (GND), U14024.7 (GND), U14025.7 (GND), U14025.7 (GND), U14025.7 (GND), U14025.7 (GND), U14026.7 (GND), U14026.7 (GND), U14027.7 (GND), U14027.7 (GND), U14027.7 (GND), U14027.7 (GND), U14028.7 (GND), U14028.7 (GND), U14028.7 (GND), U14028.7 (GND), U14028.7 (GND), U14028.7 (GND), U14029.7 (GND), U14029.7 (GND), U14029.7 (GND), U14030.7 (GND), U14030.7 (GND), U14030.7 (GND), U14030.7 (GND), U14031.7 (GND), U14031.7 (GND), U14031.7 (GND), U14032.7 (GND), U14033.7 (GND), U14033.7 (GND), U14060.7 (GND)
- net GOJ1: now also U14026.10
- net GOJAM: now also U14021.11, U14021.13, U14024.10, U14024.4, U14029.3, U14032.13
- net MP1: now also U14026.11
- net PHS3/: now also U14021.4, U14023.5, U14027.6, U14030.12, U14031.6
- net PHS4/: now also U14022.12, U14023.13, U14029.13
- net S11: now also U14026.3
- net S12: now also U14026.4
- net T01: now also U14024.2
- net T02/: now also U14022.11
- net T05/: now also U14020.11, U14030.11, U14031.5
- net T10/: now also U14022.6, U14023.1, U14023.4
- net T12A: now also U14021.10
- net TCSAJ3: now also U14026.2
- net TIMR: now also U14023.9, U14024.1
- net TPGF: now also U14031.8
- net VCC: now also R14003.1, R14004.1, U14012.14 (VCC), U14014.14 (VCC), U14014.14 (VCC), U14020.14 (VCC), U14021.14 (VCC), U14021.14 (VCC), U14021.14 (VCC), U14022.14 (VCC), U14022.14 (VCC), U14022.14 (VCC), U14022.14 (VCC), U14023.14 (VCC), U14023.14 (VCC), U14023.14 (VCC), U14024.14 (VCC), U14024.14 (VCC), U14024.14 (VCC), U14025.14 (VCC), U14025.14 (VCC), U14025.14 (VCC), U14025.14 (VCC), U14026.14 (VCC), U14026.14 (VCC), U14027.14 (VCC), U14027.14 (VCC), U14027.14 (VCC), U14027.14 (VCC), U14028.14 (VCC), U14028.14 (VCC), U14028.14 (VCC), U14028.14 (VCC), U14028.14 (VCC), U14028.14 (VCC), U14029.14 (VCC), U14029.14 (VCC), U14029.14 (VCC), U14030.14 (VCC), U14030.14 (VCC), U14030.14 (VCC), U14030.14 (VCC), U14031.14 (VCC), U14031.14 (VCC), U14031.14 (VCC), U14032.14 (VCC), U14033.14 (VCC), U14033.14 (VCC), U14060.14 (VCC)
- net at U14016.9, U14017.10: now also U14060.3
- net at U14020.3: now also U14023.12
- net at U14020.6: now also U14022.9, U14023.6
- new net: U14021.1, U14025.13, U14027.3
- new net: U14021.12, U14025.12
- new net: U14021.2, U14027.4
- new net: U14021.6, U14027.8
- new net: U14014.11, U14026.1
- new net: U14014.13, U14026.13
- new net: U14020.13, U14022.2
- new net: U14021.8, U14022.3
- new net: U14022.10, U14023.11, U14028.9
- new net: U14022.4, U14025.3
- new net: U14022.13, U14023.10
- new net: U14022.8, U14023.8
- new net: U14024.12, U14025.2
- new net: U14024.13, U14025.1, U14025.5
- new net: U14025.10, U14025.11
- new net: U14024.3, U14027.10, U14028.1
- new net: U14024.6, U14027.9
- new net: U14027.11, U14029.12
- new net: U14024.8, U14027.12
- new net: U14024.9, U14027.13, U14028.3
- new net: U14030.2, U14030.4, U14030.8
- new net: U14030.13, U14030.5
- new net: U14030.10, U14030.6
- new net: U14028.5, U14029.5, U14031.1
- new net: U14032.12, U14033.1
- new net: U14031.4, U14033.3
- new net CHINC: U14026.9
- new net ERAS: R14003.2, U14012.13, U14014.10, U14014.12
- new net ERAS/: U14012.12, U14020.12, U14021.3, U14025.8, U14029.1, U14029.10, U14032.2
- new net FNERAS/: U14021.9, U14022.1, U14022.5, U14023.2, U14023.3
- new net INOUT: U14026.5
- new net MAMU: U14026.12
- new net REDRST: U14024.11, U14024.5, U14030.1
- new net REX: U14028.4
- new net REY: U14028.2
- new net RSTK/: U14028.11, U14028.13, U14028.8
- new net RSTKX/: U14028.12
- new net RSTKY/: U14028.10
- new net SBE: U14028.6
- new net SBESET: U14029.8, U14031.3
- new net SCAD: U14029.11, U14032.1
- new net SETEK: U14027.1
- new net STBE: U14029.6, U14031.2
- new net STRT2: U14025.6, U14027.2, U14060.2
- new net T03/: U14021.5, U14025.9, U14029.2
- new net T04/: U14029.9
- new net T05: U14029.4, U14030.3
- new net T06: U14030.9
- new net T06/: U14027.5
- new net TPARG/: U14031.10
- new net TPGE: R14004.2, U14031.9, U14033.2, U14033.4
- new net ZID: U14025.4
Other:
- moved on the sheet: U14008E, U14008F, U14010A, U14010B, U14010C, U14010D, U14012D, U14012E, U14017D, U14018A, U14018B, U14018C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

Commit message: Lots of initial conditions, some missed gates, and some wiring fixes
Parts:
- U14009: Initial 1 -> (none)
- U14011: Initial (none) -> 1
Changed lines of the file:
@@
 F 2 "" H 4400 5700 60  0000 C CNN
 F 3 "" H 4400 5700 60  0000 C CNN
-F 4 "1" H 4650 5700 60  0000 C CIN "Initial"
 	3    4400 5700
 	1    0    0    -1
@@
 F 2 "" H 4400 6400 60  0000 C CNN
 F 3 "" H 4400 6400 60  0000 C CNN
+F 4 "1" H 4650 6400 60  0000 C CIN "Initial"
 	1    4400 6400
 	1    0    0    -1
@@
 $EndComp
 $Comp
-L VCC #PWR05
+L VCC #PWR04
 U 1 1 56BBFEA9
 P 3500 6150
-F 0 "#PWR05" H 3500 6000 50  0001 C CNN
+F 0 "#PWR04" H 3500 6000 50  0001 C CNN
 F 1 "VCC" H 3500 6300 50  0000 C CNN
 F 2 "" H 3500 6150 60  0000 C CNN
@@
 $EndComp
 $Comp
-L VCC #PWR06
+L VCC #PWR05
 U 1 1 56BC3D98
 P 3500 7900
-F 0 "#PWR06" H 3500 7750 50  0001 C CNN
+F 0 "#PWR05" H 3500 7750 50  0001 C CNN
 F 1 "VCC" H 3500 8050 50  0000 C CNN
 F 2 "" H 3500 7900 60  0000 C CNN
@@
 $EndComp
 $Comp
-L VCC #PWR07
+L VCC #PWR06
 U 1 1 56BF383A
 P 17750 5100
-F 0 "#PWR07" H 17750 4950 50  0001 C CNN
+F 0 "#PWR06" H 17750 4950 50  0001 C CNN
 F 1 "VCC" H 17750 5250 50  0000 C CNN
 F 2 "" H 17750 5100 60  0000 C CNN
@@
 $EndComp
 $Comp
-L VCC #PWR08
+L VCC #PWR07
 U 1 1 56CD83C7
 P 21200 13100
-F 0 "#PWR08" H 21200 12950 50  0001 C CNN
+F 0 "#PWR07" H 21200 12950 50  0001 C CNN
 F 1 "VCC" H 21200 13250 50  0000 C CNN
 F 2 "" H 21200 13100 60  0000 C CNN

Commit message: Fixed not->1-input nor in the rest of the modules.
Other:
- moved on the sheet: R14002, R14003, R14004, U14003A, U14003B, U14003C, U14003D, U14003E, U14003F, U14008A, U14008B, U14008C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

Commit message: Updated Memory Timing and Addressing to be on +4VSW
Connections:
- net labels added: +4VSW
- net labels removed: VCC

Commit message: Changed STRT2 to MYCLMP in module A14, per ND-1021042. Apparently there are *two* signals named STRT2 in the AGC, and the schematics don't differentiate them.
Connections:
- net labels added: MYCLMP
- net labels removed: STRT2
Changed lines of the file:
@@
 LIBS:valves
 LIBS:memory_timing_addressing-cache
-EELAYER 25 0
+EELAYER 26 0
 EELAYER END
 $Descr A1 33110 23386
@@
 $EndComp
 Text HLabel 29050 7250 0    60   Input ~ 0
-STRT2
+MYCLMP
 Text HLabel 30500 7150 2    60   Output ~ 0
 ZID
@@
 	7250 9050 7200 9050
 Text HLabel 7200 9050 0    60   Input ~ 0
-STRT2
+MYCLMP
 $Comp
 L +4VSW #PWR010
