File: inout_iv/a19_1.sch (KiCad schematic (older format))
At the start: 33 parts, among them U19001 74HC02, U19002 74HC04, U19003 74HC27, U19004 74HC02, U19005 74HC02, U19006 74HC02, U19007 74HC02, U19008 74HC27, U19009 74HC02, U19010 74HC02, U19011 74HC27, U19012 74HC02, U19013 74HC02, U19014 74HC27, U19015 74HC02, U19016 74HC04, U19017 74HC27, U19018 74HC02, U19019 74HC4002, U19020 74HC02, U19021 74HC02, U19022 74HC02, U19023 74HC02, U19024 74HC27, U19025 74HC02, U19026 74HC02, U19027 74HC02, U19028 74HC02, U19029 74HC02, U19030 74HC27, U19031 74HC02, U19032 74HC02, U19033 74HC04

Commit message: Tied in Inout IV and renamed MONPCH to the original MON+CH
Parts:
- U19002, U19016, U19018, U19033: Initial (none) -> 1
Connections:
- net CCH33: now reaches U19024.2, U19024.6
- net at U19026.8, U19027.3, U19027.9: now also U19024.9, U19025.13, U19026.6; no longer U19024.8, U19025.12
- net at U19029.10, U19029.12, U19030.1: now also U19031.2, U19031.9, U19032.3
- new net: U19024.8, U19025.12
- new net: U19029.9, U19030.12
Other:
- moved on the sheet: U19024B, U19026C, U19026D, U19027A, U19027B, U19027C, U19027D, U19028A, U19031A, U19031B, U19031C, U19031D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

Commit message: Fixed not->1-input nor in the rest of the modules.
Other:
- moved on the sheet: U19002A, U19002B, U19002C, U19002D, U19002E, U19002F, U19008C, U19015A, U19015B, U19016A, U19016B, U19016C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

Commit message: This adds fixes to the schematics for changes identified in comparing against the independent AGC schematics in the "schematics" branch of the main Virtual AGC repository.  Changes include:  Topological (but not logical) fixes to the DKCTR4,5,4/,5/ signals in the inout_v schematic. Wiring fix (incorrect signal sources for 5 gates) in inout_iv. Fixed incorrect signal source (including MGOJAM output polarity) for one gate in timer.  Fixed incorrect topology (but not logic) for 3 output signals in service_gates. Fixed backplane signal source (MYCLMP incorrectly used everywhere in place of the correct STRT2) in memory_timing_addressing.  ROPER, ROPES, ROPET had incorrectly omitted STRT2 as an input signal in four_bit_2. A couple of  internal nets local to sheets were also renamed due to conflicts with analysis software.  None of these fixes had any measurable effect on instruction execution; Validation was passed prior to the fixes, and continues to be passed after the fixes, and the identical instruction sequence occurs in doing so.
For me, warnings about missing components from the libraries occur upon every schematic load, though
these missing components don't seem to actually be in the circuits.  I tried to make some library
changes to work around that.  My changes don't actually fix the problem, but rather than try to back
them out and redo all the testing, they're a part of this commit as well.
Connections:
- net labels added: RCH13/
Changed lines of the file:
@@
 LIBS:valves
 LIBS:inout_iv-cache
-EELAYER 25 0
+EELAYER 26 0
 EELAYER END
 $Descr A2 23386 16535
@@
 Connection ~ 13950 4000
 Text HLabel 14300 4200 0    60   Input ~ 0
-CCH13
+RCH13/
 Wire Wire Line
 	14300 4200 14400 4200
