File: rupt_service/a15_1.sch (KiCad schematic (older format))
At the start: 27 parts, among them U15001 74HC02, U15002 74HC27, U15003 74HC04, U15004 74LVC07, U15005 74HC27, U15006 74HC02, U15007 74HC02, U15008 74HC27, U15009 74HC02, U15010 74HC27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

Commit message: Fixed not->1-input nor in the rest of the modules.
Connections:
- wire segments 370 -> 372
Other:
- moved on the sheet: U15003A, U15003B, U15003C, U15003D, U15003E, U15003F, U15004A, U15004B, U15004C, U15004D, U15004E, U15004F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
